File: IREC2025_FlightComputer/IREC2025_FlightComputer.kicad_pcb (KiCad board)
At the start: 2 copper layers, 0 parts

Commit message: update
21/3/2025
Parts:
- added BT1: Battery, Battery:BatteryHolder_Seiko_MS621F, F.Cu at (145.9, 88.5)
- added C1: 100pF, PCM_JLCPCB:C_0402, F.Cu at (107.1, 87.0)
- added C10: 100nF, PCM_JLCPCB:C_0402, F.Cu at (110.0, 88.8)
- added C11: 100nF, PCM_JLCPCB:C_0402, F.Cu at (110.0, 90.7)
- added C12: 1uF, PCM_JLCPCB:C_0402, F.Cu at (110.0, 92.5)
- added C13: 100nF, PCM_JLCPCB:C_0402, F.Cu at (110.0, 94.3)
- added C14: 10nF, PCM_JLCPCB:C_0402, F.Cu at (110.0, 96.2)
- added C15: 1uF, PCM_JLCPCB:C_0402, F.Cu at (110.0, 98.0)
- added C16: 1uF, PCM_JLCPCB:C_0402, F.Cu at (110.0, 99.9)
- added C17: 100nF, PCM_JLCPCB:C_0402, F.Cu at (112.8, 87.0)
- added C18: 10uF, PCM_JLCPCB:C_0402, F.Cu at (112.8, 88.8)
- added C19: 100nF, PCM_JLCPCB:C_0402, F.Cu at (112.8, 90.7)
- added C2: 100nF, PCM_JLCPCB:C_0402, F.Cu at (107.1, 88.8)
- added C20: 10uF, PCM_JLCPCB:C_0603, F.Cu at (132.2, 101.0)
- added C21: 2.2uF, PCM_JLCPCB:C_0402, F.Cu at (112.8, 92.5)
- added C23: RVT1E101M0607, EasyEDA:CAP-SMD_BD6.3-L6.6-W6.6-LS7.2-R-RD, F.Cu at (128.9, 71.5)
- added C25: 3.3pF, PCM_JLCPCB:C_0402, F.Cu at (112.8, 94.3)
- added C26: 4.7uF, PCM_JLCPCB:C_0402, F.Cu at (112.8, 96.2)
- added C27: 22uF, PCM_JLCPCB:C_0805, F.Cu at (131.9, 84.0)
- added C28: 100uF, PCM_JLCPCB:C_CASE-B-3528-21(mm), F.Cu at (102.3, 101.0)
- added C29: 3.0pF, PCM_JLCPCB:C_0402, F.Cu at (138.1, 95.6)
- added C3: 1uF, PCM_JLCPCB:C_0402, F.Cu at (107.1, 90.7)
- added C30: 47nF, PCM_JLCPCB:C_0402, F.Cu at (138.1, 97.5)
- added C31: 47pF, PCM_JLCPCB:C_0402, F.Cu at (138.1, 99.3)
- added C32: 47pF, PCM_JLCPCB:C_0402, F.Cu at (138.1, 101.2)
- added C33: C_Small, PCM_JLCPCB:C_0402, F.Cu at (138.1, 103.0)
- added C34: 1uF, PCM_JLCPCB:C_0402, F.Cu at (138.1, 104.9)
- added C35: 100nF, PCM_JLCPCB:C_0402, F.Cu at (141.0, 95.6)
- added C36: C_Small, PCM_JLCPCB:C_0402, F.Cu at (141.0, 97.5)
- added C37: C_Small, PCM_JLCPCB:C_0402, F.Cu at (141.0, 99.3)
- added C38: C_Small, PCM_JLCPCB:C_0402, F.Cu at (141.0, 101.2)
- added C39: C_Small, PCM_JLCPCB:C_0402, F.Cu at (141.0, 103.0)
- added C4: 10uF, PCM_JLCPCB:C_0402, F.Cu at (107.1, 92.5)
- added C40: C_Small, PCM_JLCPCB:C_0402, F.Cu at (141.0, 104.9)
- added C41: 10nF, PCM_JLCPCB:C_0402, F.Cu at (143.8, 95.6)
- added C42: C_Small, PCM_JLCPCB:C_0402, F.Cu at (143.8, 97.5)
- added C43: 470nF, PCM_JLCPCB:C_0402, F.Cu at (143.8, 99.3)
- added C44: 1uF, PCM_JLCPCB:C_0402, F.Cu at (143.8, 101.2)
- added C45: 100nF, PCM_JLCPCB:C_0402, F.Cu at (143.8, 103.0)
- added C46: C_Small, PCM_JLCPCB:C_0402, F.Cu at (143.8, 104.9)
- added C47: C_Small, PCM_JLCPCB:C_0402, F.Cu at (146.7, 95.6)
- added C48: C_Small, PCM_JLCPCB:C_0402, F.Cu at (146.7, 97.5)
- added C49: 10nF, PCM_JLCPCB:C_0402, F.Cu at (146.7, 99.3)
- added C5: 100nF, PCM_JLCPCB:C_0402, F.Cu at (107.1, 94.3)
- added C50: 1nF, PCM_JLCPCB:C_0402, F.Cu at (146.7, 101.2)
- added C51: 100nF, PCM_JLCPCB:C_0402, F.Cu at (138.1, 113.8)
- added C52: 10uF, PCM_JLCPCB:C_0402, F.Cu at (138.1, 115.7)
- added C53: 100nF, PCM_JLCPCB:C_0402, F.Cu at (138.1, 117.5)
- added C54: 1uF, PCM_JLCPCB:C_0402, F.Cu at (138.1, 119.4)
- added C55: 10uF, PCM_JLCPCB:C_0402, F.Cu at (138.1, 121.2)
- added C56: 100nF, PCM_JLCPCB:C_0402, F.Cu at (141.0, 113.8)
- added C57: 100nF, PCM_JLCPCB:C_0402, F.Cu at (141.0, 115.7)
- added C58: 100nF, PCM_JLCPCB:C_0402, F.Cu at (141.0, 117.5)
- added C59: 100nF, PCM_JLCPCB:C_0402, F.Cu at (141.0, 119.4)
- added C6: 100nF, PCM_JLCPCB:C_0402, F.Cu at (107.1, 96.2)
- added C60: 10uF, PCM_JLCPCB:C_0402, F.Cu at (95.4, 112.7)
- added C61: 10nF, PCM_JLCPCB:C_0402, F.Cu at (95.4, 114.6)
- added C62: 10nF, PCM_JLCPCB:C_0402, F.Cu at (95.4, 116.4)
- added C63: 10nF, PCM_JLCPCB:C_0402, F.Cu at (95.4, 118.3)
- added C64: 10nF, PCM_JLCPCB:C_0402, F.Cu at (95.4, 120.1)
- added C65: 10nF, PCM_JLCPCB:C_0402, F.Cu at (95.4, 122.0)
- added C66: 10nF, PCM_JLCPCB:C_0402, F.Cu at (95.4, 123.8)
- added C67: 10nF, PCM_JLCPCB:C_0402, F.Cu at (98.3, 112.7)
- added C68: 10nF, PCM_JLCPCB:C_0402, F.Cu at (98.3, 114.6)
- added C69: 10nF, PCM_JLCPCB:C_0402, F.Cu at (98.3, 116.4)
- added C7: 100nF, PCM_JLCPCB:C_0402, F.Cu at (107.1, 98.0)
- added C70: 10uF, PCM_JLCPCB:C_0402, F.Cu at (98.3, 118.3)
- added C71: 1uF, PCM_JLCPCB:C_0402, F.Cu at (156.0, 68.5)
- added C8: 100nF, PCM_JLCPCB:C_0402, F.Cu at (107.1, 99.9)
- added C9: 100nF, PCM_JLCPCB:C_0402, F.Cu at (110.0, 87.0)
- added D1: MMSZ4683T1G, EasyEDA:SOD-123_L2.8-W1.8-LS3.7-RD, F.Cu at (128.2, 107.8)
- added D2: USBLC6-2SC6, EasyEDA:SOT-23-6_L2.9-W1.6-P0.95-LS2.8-BL, F.Cu at (96.5, 106.3)
- added D3: SS34_C466502, EasyEDA:SMA_L4.4-W2.6-LS5.0-RD, F.Cu at (129.1, 104.4)
- added D4: 3v3_led, LED_SMD:LED_0805_2012Metric, F.Cu at (132.5, 95.4)
- added D6: PMEG2005EJ, Diode_SMD:D_SOD-323F, F.Cu at (153.8, 85.8)
- added FB1: 100R, PCM_JLCPCB:FB_0805, F.Cu at (101.6, 104.5)
- added J1: Molex Microfit, Connector_Molex:Molex_Micro-Fit_3.0_43650-0215_1x02_P3.00mm_Vertical, F.Cu at (98.3, 71.0)
- added JP1: U.FL-R-SMT-1(10), EasyEDA:ANT-SMD_UFL-R-SMT-1-10, F.Cu at (138.6, 108.4)
- added L1: 2.2uH,50mA, PCM_JLCPCB:L_0805, F.Cu at (101.6, 107.3)
- added L2: BLM18AG121SN1D, EasyEDA:L0603, F.Cu at (153.0, 102.0)
- added L3: 47nH, PCM_JLCPCB:C_0402, F.Cu at (146.7, 103.0)
- added L4: 0R, Inductor_SMD:L_0402_1005Metric, F.Cu at (149.6, 95.7)
- added L5: 2.5nH, PCM_JLCPCB:C_0402, F.Cu at (146.7, 104.9)
- added L6: L_Small, Inductor_SMD:L_0402_1005Metric, F.Cu at (149.6, 97.7)
- added L7: L_Small, Inductor_SMD:L_0402_1005Metric, F.Cu at (149.6, 99.7)
- added L8: 15nH, Inductor_SMD:L_0603_1608Metric, F.Cu at (153.0, 99.5)
- added L9: L_Small, Inductor_SMD:L_0402_1005Metric, F.Cu at (149.6, 101.7)
- added LED1: HS-0402-UR, EasyEDA:LED0402-R-RD, F.Cu at (149.8, 85.4)
- added LED2: HS-0402-UR, EasyEDA:LED0402-R-RD, F.Cu at (149.8, 87.8)
- added PWM1: Conn_01x03_Pin, Connector_Molex:Molex_Micro-Fit_3.0_43650-0315_1x03_P3.00mm_Vertical, F.Cu at (124.3, 89.5)
- added Pyro_A1: Molex Microfit, Connector_Molex:Molex_Micro-Fit_3.0_43650-0215_1x02_P3.00mm_Vertical, F.Cu at (98.3, 78.8)
- added Pyro_B1: Molex Microfit, Connector_Molex:Molex_Micro-Fit_3.0_43650-0215_1x02_P3.00mm_Vertical, F.Cu at (98.3, 86.7)
- added Pyro_C1: Molex Microfit, Connector_Molex:Molex_Micro-Fit_3.0_43650-0215_1x02_P3.00mm_Vertical, F.Cu at (98.3, 94.5)
- added Q1: SI7232DN-T1-GE3, EasyEDA:POWER-1212-8_L3.3-W3.3-P0.66-LS3.3-BL, F.Cu at (127.2, 77.7)
- added Q2: SI7232DN-T1-GE3, EasyEDA:POWER-1212-8_L3.3-W3.3-P0.66-LS3.3-BL, F.Cu at (127.2, 82.3)
- added R1: 10kΩ, PCM_JLCPCB:R_0402, F.Cu at (112.8, 98.0)
- added R10: 100kΩ, PCM_JLCPCB:R_0402, F.Cu at (115.7, 96.2)
- added R11: 3.3kΩ, PCM_JLCPCB:R_0402, F.Cu at (115.7, 98.0)
- added R12: 470Ω, PCM_JLCPCB:R_0402, F.Cu at (115.7, 99.9)
- added R13: 470Ω, PCM_JLCPCB:R_0402, F.Cu at (118.5, 87.0)
- added R14: 470Ω, PCM_JLCPCB:R_0402, F.Cu at (118.5, 88.8)
- added R15: 470Ω, PCM_JLCPCB:R_0402, F.Cu at (118.5, 90.7)
- added R16: 3.3kΩ, PCM_JLCPCB:R_0402, F.Cu at (118.5, 92.5)
- added R17: 3.3kΩ, PCM_JLCPCB:R_0402, F.Cu at (118.5, 94.3)
- added R18: 1k, Resistor_SMD:R_0402_1005Metric, F.Cu at (149.6, 103.7)
- added R19: 4.7kΩ, PCM_JLCPCB:R_0402, F.Cu at (141.0, 121.2)
- added R2: 47kΩ, PCM_JLCPCB:R_0402, F.Cu at (112.8, 99.9)
- added R20: 4.7kΩ, PCM_JLCPCB:R_0402, F.Cu at (143.8, 113.8)
- added R21: 2.2kΩ, PCM_JLCPCB:R_0402, F.Cu at (143.8, 115.7)
- added R22: 2.2kΩ, PCM_JLCPCB:R_0402, F.Cu at (143.8, 117.5)
- added R23: 22kΩ, PCM_JLCPCB:R_0402, F.Cu at (98.3, 120.1)
- added R24: 22kΩ, PCM_JLCPCB:R_0402, F.Cu at (98.3, 122.0)
- added R25: 22kΩ, PCM_JLCPCB:R_0402, F.Cu at (98.3, 123.8)
- added R26: 22kΩ, PCM_JLCPCB:R_0402, F.Cu at (101.1, 112.7)
- added R27: 22kΩ, PCM_JLCPCB:R_0402, F.Cu at (101.1, 114.6)
- added R28: 22kΩ, PCM_JLCPCB:R_0402, F.Cu at (101.1, 116.4)
- added R29: 22kΩ, PCM_JLCPCB:R_0402, F.Cu at (101.1, 118.3)
- added R3: 5.1kΩ, PCM_JLCPCB:R_0402, F.Cu at (115.7, 87.0)
- added R30: 22kΩ, PCM_JLCPCB:R_0402, F.Cu at (101.1, 120.1)
- added R31: 47kΩ, PCM_JLCPCB:R_0402, F.Cu at (101.1, 122.0)
- added R32: 22kΩ, PCM_JLCPCB:R_0402, F.Cu at (101.1, 123.8)
- added R33: 470Ω, PCM_JLCPCB:R_0402, F.Cu at (156.0, 70.3)
- added R34: 470Ω, PCM_JLCPCB:R_0402, F.Cu at (156.0, 72.2)
- added R35: 1kΩ, PCM_JLCPCB:R_0402, F.Cu at (156.0, 74.0)
- added R36: 1kΩ, PCM_JLCPCB:R_0402, F.Cu at (156.0, 75.9)
- added R37: 3.3kΩ, PCM_JLCPCB:R_0402, F.Cu at (156.0, 77.7)
- added R4: 5.1kΩ, PCM_JLCPCB:R_0402, F.Cu at (115.7, 88.8)
- added R5: 1MΩ, PCM_JLCPCB:R_0402, F.Cu at (115.7, 90.7)
- added R6: 10kΩ, PCM_JLCPCB:R_0402, F.Cu at (115.7, 92.5)
- added R7: 22kΩ, PCM_JLCPCB:R_0402, F.Cu at (115.7, 94.3)
- added R8: 1kΩ, PCM_JLCPCB:R_0805, F.Cu at (132.5, 98.4)
- added U1: STM32U575VGTx, Package_QFP:LQFP-100_14x14mm_P0.5mm, F.Cu at (114.9, 76.8)
- added U10: PE4259-63, EasyEDA:SC-70-6_L2.2-W1.3-P0.65-LS2.1-BL, F.Cu at (153.1, 96.4)
- added U11: SX1262IMLTRT, Package_DFN_QFN:QFN-24-1EP_4x4mm_P0.5mm_EP2.6x2.6mm, F.Cu at (151.2, 107.8)
- added U12: ADXL375BCCZ-RL7, EasyEDA:LGA-14_L5.0-W3.0-P0.80-BL, F.Cu at (140.3, 125.0)
- added U13: MMC5983MA, EasyEDA:LGA-16_L3.0-W3.0-P0.50-BL_SQ, F.Cu at (152.2, 122.0)
- added U14: BMI088, EasyEDA:LGA-16_L4.5-W3.0-P0.50-BL, F.Cu at (152.3, 115.8)
- added U15: TMP275AIDGKR VSSOP8, EasyEDA:VSSOP-8_L3.0-W3.0-P0.65-LS5.0-BL, F.Cu at (147.7, 116.4)
- added U16: MS5607-02BA, Package_LGA:LGA-8_3x5mm_P1.25mm, F.Cu at (147.7, 123.3)
- added U17: KLM4G1FETE-B041, EasyEDA:FBGA-153_L11.0-W10.0-P0.50_KLM4G1FETE-B041, F.Cu at (108.8, 117.5)
- added U18: SAM-M10Q-00B, EasyEDA:LCC-20_L15.5-W15.5-P1.90_SAM-M10Q-00B, F.Cu at (146.2, 75.9)
- added U2: NRVB120VLSFT1G, EasyEDA:SOD-123_L2.7-W1.6-LS3.7-RD-1, F.Cu at (122.7, 103.9)
- added U4: NRVB120VLSFT1G, EasyEDA:SOD-123_L2.7-W1.6-LS3.7-RD-1, F.Cu at (122.7, 106.8)
- added U5: LP5912Q3.3DRVRQ1, EasyEDA:WSON-6_L2.0-W2.0-P0.65-TL-EP, F.Cu at (132.0, 80.8)
- added U8: TPS62153, Package_DFN_QFN:VQFN-16-1EP_3x3mm_P0.5mm_EP1.68x1.68mm_ThermalVias, F.Cu at (96.7, 101.5)
- added U9: SN74HCT125DR, EasyEDA:SOIC-14_L8.7-W3.9-P1.27-LS6.0-BL, F.Cu at (125.3, 98.1)
- added USB1: 10172013-00011LF, EasyEDA:USB-C-SMD_10174570-00A11LF, F.Cu at (112.4, 104.5)
- added X1: 1XXD32000MBA, EasyEDA:OSC-SMD_4P-L2.0-W1.6-BL_1XXD, F.Cu at (131.9, 77.0)
- added X2: 1XXD32000MBA, EasyEDA:OSC-SMD_4P-L2.0-W1.6-BL_1XXD, F.Cu at (143.4, 107.4)
