File: IREC2025_FlightComputer/Miscs.kicad_sch (KiCad schematic)
At the start: 0 parts

Commit message: Schematics
Parts:
- added C43, C44, C45, C46, C47, C48, C49, C50: 10nF, PCM_JLCPCB:C_0402, symbol PCM_JLCPCB-Capacitors:0402,10nF
- added C51: 10uF, PCM_JLCPCB:C_0402, symbol PCM_JLCPCB-Capacitors:0402,10uF
- added R11: 47kΩ, PCM_JLCPCB:R_0402, symbol PCM_JLCPCB-Resistors:0402,47kΩ
- added R12, R13, R14, R15, R16, R17, R18, R19, R20: 22kΩ, PCM_JLCPCB:R_0402, symbol PCM_JLCPCB-Resistors:0402,22kΩ
- added U9: KLM4G1FETE-B041, EasyEDA:FBGA-153_L11.0-W10.0-P0.50_KLM4G1FETE-B041, symbol EasyEDA:KLM4G1FETE-B041
Connections:
- new net: R20.1, U9.H5 (DataStrobe)
- new net +3V3: C43.1, C44.1, C45.1, C46.1, C47.1, C48.1, C49.1, C50.1, C51.1, R11.2, R12.1, R13.1, R14.1, R15.1, R16.1, R17.1, R18.1, R19.1, U9.C2 (VDDI), U9.C6 (VCCQ), U9.E6 (VCC), U9.F5 (VCC), U9.J10 (VCC), U9.K9 (VCC), U9.M4 (VCCQ), U9.N4 (VCCQ), U9.P3 (VCCQ), U9.P5 (VCCQ)
- new net DAT0: R12.2, U9.A3 (DAT0)
- new net DAT1: R13.2, U9.A4 (DAT1)
- new net DAT2: R14.2, U9.A5 (DAT2)
- new net DAT3: R15.2, U9.B2 (DAT3)
- new net DAT4: R16.2, U9.B3 (DAT4)
- new net DAT5: R17.2, U9.B4 (DAT5)
- new net DAT6: R18.2, U9.B5 (DAT6)
- new net DAT7: R19.2, U9.B6 (DAT7)
- new net GND: C43.2, C44.2, C45.2, C46.2, C47.2, C48.2, C49.2, C50.2, C51.2, R20.2, U9.A6 (VSS), U9.C4 (VSS), U9.E7 (VSS), U9.G5 (VSS), U9.H10 (VSS), U9.J5 (VSS), U9.K8 (VSS), U9.N2 (VSS), U9.N5 (VSS), U9.P4 (VSS), U9.P6 (VSS)
- new net RST_n: U9.K5 (RSTN)
- new net eMMC_CLK: U9.M6 (CLK)
- new net eMMC_CMD: R11.1, U9.M5 (CMD)
- no-connect marks 0 -> 119
Other:
- note added: "eMMC"
- note added: "eMMC decoupling"

Commit message: update
21/3/2025
Parts:
- added C69: 10nF, PCM_JLCPCB:C_0402, symbol PCM_JLCPCB-Capacitors:0402,10nF
- added C70: 10uF, PCM_JLCPCB:C_0402, symbol PCM_JLCPCB-Capacitors:0402,10uF
- renumbered C51 to C60, C43 to C61, C44 to C62, C45 to C63, C46 to C64, C47 to C65, C48 to C66, C49 to C67, C50 to C68, R12 to R23, R13 to R24, R14 to R25, R15 to R26, R16 to R27, R17 to R28, R18 to R29, R19 to R30, R11 to R31, R20 to R32, U9 to U17
Connections:
- net +3V3: now also C69.1; no longer U17.C2 (VDDI)
- net GND: now also C69.2, C70.2
- new net: C70.1, U17.C2 (VDDI)
