File: IREC2025_FlightComputer/Sensors.kicad_sch (KiCad schematic)
At the start: 5 parts, among them U6 ADXL375BCCZ-RL7, U7 BMI088

Commit message: Schematics
Parts:
- added C57, C58, C63, C64: 100nF, PCM_JLCPCB:C_0402, symbol PCM_JLCPCB-Capacitors:0402,100nF
- added C59: 1uF, PCM_JLCPCB:C_0402, symbol PCM_JLCPCB-Capacitors:0402,1uF
- added C60: 10uF, PCM_JLCPCB:C_0402, symbol PCM_JLCPCB-Capacitors:0402,10uF
- added R23, R24: 4.7kΩ, PCM_JLCPCB:R_0402, symbol PCM_JLCPCB-Resistors:0402,4.7kΩ
- added R26, R27: 2.2kΩ, PCM_JLCPCB:R_0402, symbol PCM_JLCPCB-Resistors:0402,2.2kΩ
- added U12: MMC5983MA, EasyEDA:LGA-16_L3.0-W3.0-P0.50-BL_SQ, symbol EasyEDA:MMC5983MA
- added U16: TMP275AIDGKR VSSOP8, EasyEDA:VSSOP-8_L3.0-W3.0-P0.65-LS5.0-BL, symbol EasyEDA:TMP275AIDGKRVSSOP8
- added U17: MS5607-02BA, Package_LGA:LGA-8_3x5mm_P1.25mm, symbol Sensor_Pressure:MS5607-02BA
Connections:
- net +3.3V: now also U7.11 (VDDIO), U7.3 (VDD), C57.1, C58.1, C59.1, C63.1, C64.2, R23.1, R24.2, R26.1, R27.1, U12.13 (VDDIO), U12.2 (VDD), U16.8 (V+), U17.1 (VDD)
- net ADXL_INT1: no longer U7.1 (INT2)
- net GND: now also U7.2 (NC), U7.4 (GNDA), U7.7 (PS), C57.2, C58.2, C59.2, C60.2, C63.2, C64.1, U12.11 (GND), U12.9 (GND), U16.4 (GND), U16.5 (A2), U16.6 (A1), U16.7 (A0), U17.2 (PS), U17.3 (GND)
- net BMI_accel_CS: now reaches U7.14 (CSB1)
- net BMI_accel_INT: now reaches U7.16 (INT1)
- net BMI_accel_INT: now also U7.1 (INT2)
- net BMI_SCLK: now reaches U7.8 (SCL/SCK)
- new net: C60.1, U12.10 (CAP)
- new net MMC_INT: U12.15 (INT)
- new net MMC_SCL: R23.2, U12.1 (SCL/SPI_SCK)
- new net MMC_SDA: R24.1, U12.16 (SDA/SPI_SDI)
- new net MS5607_CS: U17.4 (CSB), U17.5 (CSB)
- new net MS5607_MISO: U17.6 (SDO)
- new net MS5607_MOSI: U17.7 (SDI/SDA)
- new net MS5607_SCLK: U17.8 (SCLK)
- new net TMP_ALERT: U16.3 (ALERT)
- new net TMP_SCL: R26.2, U16.2 (SCL)
- new net TMP_SDA: R27.2, U16.1 (SDA)
- no-connect marks 2 -> 10
Other:
- note added: "ADXL375BCCZ-RL7 (High-G) SPI (Dedicated bus)"
- note added: "Altimeter SPI"
- note added: "BMI088 (Low-G) SPI"
- note added: "MMC5983MA Magnetometer I2C"
- note added: "Shared SPI Bus (SPI3)"
- note added: "TMP275 I2C"
- note removed: "ADXL375BCCZ-RL7 (High-G)"
- note removed: "SPI"
- moved on the sheet: C40, C41, C42, U6, U7

Commit message: update
21/3/2025
Parts:
- renumbered C40 to C51, C42 to C52, C41 to C53, C59 to C54, C60 to C55, C63 to C56, C64 to C59, R24 to R19, R23 to R20, R27 to R21, R26 to R22, U6 to U12, U12 to U13, U7 to U14, U16 to U15, U17 to U16
Connections:
- net ADXL_CS renamed ADXL_NSS
- net BMI_GYRO_INT renamed BMI_GYRO_INT1
- net BMI_GYRO_INT1: no longer U14.13 (INT4)
- net BMI_accel_INT renamed BMI_accel_INT1
- net BMI_accel_INT1: no longer U14.1 (INT2)
- new net BMI_GYRO_INT2: U14.13 (INT4)
- new net BMI_accel_INT2: U14.1 (INT2)

Commit message: Updated 22/3/2025
Connections:
- net MS5607_CS renamed MS5607_NSS
Changed lines of the file:
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@@
 		)
 	)
-	(global_label "MS5607_CS"
+	(global_label "MS5607_NSS"
 		(shape input)
 		(at 34.29 175.26 180)
@@
 		)
 		(property "Intersheetrefs" "${INTERSHEET_REFS}"
-			(at 20.3588 175.26 0)
+			(at 19.0888 175.26 0)
 			(effects
 				(font

Commit message: update idk
25/3/2025
starting to take shape (i guess)
Connections:
- net +3.3V: now also U12.1 (VDDI/O)
- net GND: no longer U12.1 (VDDI/O)
Other:
- moved on the sheet: C51

Commit message: checkpoint
before the great layout change
Connections:
- net GND: now also U14.6 (GNDIO)
Other:
- note added: "CL21B106KOQNNNE"
- note added: "ERJ-2RKF2201X"
- note added: "GRM155R70J105KA12D"
- note added: "GRM155R71H104KE14D"
- note added: "RC0402JR-074K7L"
Changed lines of the file:
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@@
 		)
 	)
+	(text "	\nERJ-2RKF2201X"
+		(exclude_from_sim no)
+		(at 167.64 93.472 90)
+		(effects
+			(font
+				(size 0.635 0.635)
+			)
+		)
+	)
+	(text "CL21B106KOQNNNE"
+		(exclude_from_sim no)
+		(at 235.204 57.912 0)
+		(effects
+			(font
+				(size 0.635 0.635)
+			)
+		)
+	)
+	(text "GRM155R71H104KE14D"
+		(exclude_from_sim no)
+		(at 116.078 112.014 0)
+		(effects
+			(font
+				(size 0.635 0.635)
+			)
+		)
+	)
+	(text "GRM155R71H104KE14D"
+		(exclude_from_sim no)
+		(at 230.886 106.68 0)
+		(effects
+			(font
+				(size 0.635 0.635)
+			)
+		)
+	)
+	(text "RC0402JR-074K7L"
+		(exclude_from_sim no)
+		(at 236.22 33.782 0)
+		(effects
+			(font
+				(size 0.635 0.635)
+			)
+		)
+	)
+	(text "RC0402JR-074K7L"
+		(exclude_from_sim no)
+		(at 169.926 37.592 0)
+		(effects
+			(font
+				(size 0.635 0.635)
+			)
+		)
+	)
+	(text "GRM155R70J105KA12D"
+		(exclude_from_sim no)
+		(at 163.83 48.26 0)
+		(effects
+			(font
+				(size 0.635 0.635)
+			)
+		)
+	)
 	(text "TMP275 I2C"
 		(exclude_from_sim no)
@@
 		)
 	)
+	(text "	\nERJ-2RKF2201X"
+		(exclude_from_sim no)
+		(at 176.784 93.472 90)
+		(effects
+			(font
+				(size 0.635 0.635)
+			)
+		)
+	)
 	(text "MMC5983MA Magnetometer I2C"
 		(exclude_from_sim no)
@@
 		)
 	)
+	(text "CL21B106KOQNNNE"
+		(exclude_from_sim no)
+		(at 31.242 47.498 0)
+		(effects
+			(font
+				(size 0.635 0.635)
+			)
+		)
+	)
+	(text "GRM155R71H104KE14D"
+		(exclude_from_sim no)
+		(at 49.276 155.448 0)
+		(effects
+			(font
+				(size 0.635 0.635)
+			)
+		)
+	)
+	(text "GRM155R71H104KE14D"
+		(exclude_from_sim no)
+		(at 42.926 47.498 0)
+		(effects
+			(font
+				(size 0.635 0.635)
+			)
+		)
+	)
+	(text "GRM155R71H104KE14D"
+		(exclude_from_sim no)
+		(at 34.29 109.982 0)
+		(effects
+			(font
+				(size 0.635 0.635)
+			)
+		)
+	)
 	(text "ADXL375BCCZ-RL7 (High-G) SPI (Dedicated bus)"
 		(exclude_from_sim no)
@@
 		)
 	)
+	(text "GRM155R71H104KE14D"
+		(exclude_from_sim no)
+		(at 37.592 34.798 0)
+		(effects
+			(font
+				(size 0.635 0.635)
+			)
+		)
+	)
 	(text_box "SPI1: SX1262 LoRa\nSPI2: ADXL375BCCZ-RL7\nSPI3: BMI088 and MS5207"
 		(exclude_from_sim no)
@@
 	)
 	(junction
+		(at 44.45 101.6)
+		(diameter 0)
+		(color 0 0 0 0)
+	)
+	(junction
 		(at 175.26 35.56)
 		(diameter 0)
@@
 	(wire
 		(pts
+			(xy 44.45 101.6) (xy 46.99 101.6)
+		)
+		(stroke
+			(width 0)
+			(type default)
+		)
+	)
+	(wire
+		(pts
 			(xy 60.96 182.88) (xy 36.83 182.88)
 		)
@@
 	(wire
 		(pts
+			(xy 44.45 101.6) (xy 44.45 96.52)
+		)
+		(stroke
+			(width 0)
+			(type default)
+		)
+	)
+	(wire
+		(pts
 			(xy 90.17 99.06) (xy 113.03 99.06)
 		)
@@
 	(wire
 		(pts
-			(xy 44.45 104.14) (xy 44.45 96.52)
+			(xy 44.45 104.14) (xy 44.45 101.6)
 		)
 		(stroke
@@
 				)
 				(justify left)
+				(hide yes)
 			)
 		)
@@
 					(size 0.8 0.8)
 				)
+				(hide yes)
 			)
 		)
@@
 				)
 				(justify left)
+				(hide yes)
 			)
 		)
@@
 					(size 0.8 0.8)
 				)
+				(hide yes)
 			)
 		)
@@
 				)
 				(justify left)
+				(hide yes)
 			)
 		)
@@
 				)
 				(justify left)
+				(hide yes)
 			)
 		)
@@
 				)
 				(justify left)
+				(hide yes)
 			)
 		)
@@
 				)
 				(justify left)
+				(hide yes)
 			)
 		)

Commit message: 2 designs
Parts:
- added C62: 10uF, PCM_JLCPCB:C_0402, symbol PCM_JLCPCB-Capacitors:0402,10uF
- added C63, C64: 100nF, PCM_JLCPCB:C_0402, symbol PCM_JLCPCB-Capacitors:0402,100nF
- added U17: ADXL375BCCZ-RL7, EasyEDA:LGA-14_L5.0-W3.0-P0.80-BL, symbol EasyEDA:ADXL375BCCZ-RL7
- renumbered C51 to C?, C59 to C?, C54 to C?, C55 to C?, C56 to C?, C52 to C?, C57 to C?, R22 to R?, R20 to R?, U15 to U?, U13 to U?, U16 to U?, U14 to U?
Connections:
- net +3.3V: now also C62.2, C63.1, C64.2, U17.1 (VDDI/O), U17.6 (VS)
- net ADXL_INT1: now also U17.8 (INT1)
- net ADXL_INT2: now also U17.9 (INT2)
- net ADXL_MISO: now also U17.12 (SDO/ALTADDRESS)
- net ADXL_MOSI: now also U17.13 (SDA/SDI/SDIO)
- net ADXL_NSS: now also U17.7 (~{CS})
- net ADXL_SCLK: now also U17.14 (SCL/SCLK)
- net GND: now also C62.1, C63.2, C64.1, U17.10 (NC), U17.2 (GND), U17.4 (GND), U17.5 (GND)
- no-connect marks 10 -> 12
Other:
- note added: "ADXL375BCCZ-RL7 (Breakout)"

Commit message: changed most resistors to 0603
Parts:
- removed C62: 10uF, PCM_JLCPCB:C_0402, symbol PCM_JLCPCB-Capacitors:0402,10uF
- removed C63, C64: 100nF, PCM_JLCPCB:C_0402, symbol PCM_JLCPCB-Capacitors:0402,100nF
- removed U17: ADXL375BCCZ-RL7, EasyEDA:LGA-14_L5.0-W3.0-P0.80-BL, symbol EasyEDA:ADXL375BCCZ-RL7
- R19, R21: footprint PCM_JLCPCB:R_0402 -> PCM_JLCPCB:R_0603
- R7: renamed from R?; footprint PCM_JLCPCB:R_0402 -> PCM_JLCPCB:R_0603
- gave numbers to parts that had none: 12
Connections:
- no-connect marks 12 -> 10
Other:
- note removed: "ADXL375BCCZ-RL7 (Breakout)"
