File: IREC2025_FlightComputer/untitled.kicad_sch (KiCad schematic)
At the start: 36 parts, among them U4 PE4259-63, U5 SX1262IMLTRT, Y1 32 MHz TCXO

Commit message: Schematics
Parts:
- removed C27: C_Small, PCM_JLCPCB:C_0402, symbol Device:C_Small
- removed R11: R, Resistor_SMD:R_0402_1005Metric, symbol Device:R_Small
- C28: value C_Small -> 10nF
Connections:
- net XTA: now also Y1.3 (OUTPUT)
- net MISO renamed LoRa_MISO
- net MOSI renamed LoRa_MOSI
- net NSS renamed LoRa_NSS
- net SCK renamed LoRa_SCLK
Changed lines of the file:
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@@
 	(text "DIO1: TXDONE\n  DIO2: RF Switch\n DIO3: RXDONE "
 		(exclude_from_sim no)
-		(at 252.222 149.86 0)
+		(at 250.19 149.606 0)
 		(effects
 			(font
@@
 	(wire
 		(pts
+			(xy 100.33 40.64) (xy 104.14 40.64)
+		)
+		(stroke
+			(width 0)
+			(type default)
+		)
+	)
+	(wire
+		(pts
 			(xy 55.88 90.17) (xy 62.23 90.17)
 		)
@@
 	(wire
 		(pts
-			(xy 113.03 40.64) (xy 115.57 40.64)
-		)
-		(stroke
-			(width 0)
-			(type default)
-		)
-	)
-	(wire
-		(pts
 			(xy 283.21 123.19) (xy 283.21 127)
 		)
@@
 	(wire
 		(pts
-			(xy 107.95 40.64) (xy 105.41 40.64)
-		)
-		(stroke
-			(width 0)
-			(type default)
-		)
-	)
-	(wire
-		(pts
 			(xy 59.69 40.64) (xy 40.64 40.64)
 		)
@@
 		)
 	)
-	(global_label "MISO"
+	(global_label "LoRa_MISO"
 		(shape input)
 		(at 264.16 138.43 270)
@@
 		)
 		(property "Intersheetrefs" "${INTERSHEET_REFS}"
-			(at 264.16 146.0114 90)
+			(at 264.16 151.5751 90)
 			(effects
 				(font
@@
 	(global_label "XTA"
 		(shape input)
-		(at 115.57 40.64 0)
+		(at 104.14 40.64 0)
 		(fields_autoplaced yes)
 		(effects
@@
 		)
 		(property "Intersheetrefs" "${INTERSHEET_REFS}"
-			(at 121.8209 40.64 0)
+			(at 110.3909 40.64 0)
 			(effects
 				(font
@@
 		)
 	)
-	(global_label "SCK"
+	(global_label "LoRa_SCLK"
 		(shape input)
 		(at 261.62 138.43 270)
@@
 		)
 		(property "Intersheetrefs" "${INTERSHEET_REFS}"
-			(at 261.62 145.1647 90)
+			(at 261.62 151.7565 90)
 			(effects
 				(font
@@
 		)
 	)
-	(global_label "NSS"
+	(global_label "LoRa_NSS"
 		(shape input)
 		(at 269.24 138.43 270)
@@
 		)
 		(property "Intersheetrefs" "${INTERSHEET_REFS}"
-			(at 269.24 145.1647 90)
+			(at 269.24 150.7284 90)
 			(effects
 				(font
@@
 		)
 	)
-	(global_label "MOSI"
+	(global_label "LoRa_MOSI"
 		(shape input)
 		(at 266.7 138.43 270)
@@
 		)
 		(property "Intersheetrefs" "${INTERSHEET_REFS}"
-			(at 266.7 146.0114 90)
+			(at 266.7 151.5751 90)
 			(effects
 				(font
@@
 			)
 		)
-		(property "Value" "C_Small"
+		(property "Value" "10nF"
 			(at 43.18 58.4262 0)
 			(effects
@@
 	)
 	(symbol
-		(lib_id "Device:C_Small")
-		(at 102.87 40.64 90)
-		(unit 1)
-		(exclude_from_sim no)
-		(in_bom yes)
-		(on_board yes)
-		(dnp no)
-		(fields_autoplaced yes)
-		(property "Reference" "C27"
-			(at 102.8763 34.29 90)
-			(effects
-				(font
-					(size 1.27 1.27)
-				)
-			)
-		)
-		(property "Value" "C_Small"
-			(at 102.8763 36.83 90)
-			(effects
-				(font
-					(size 1.27 1.27)
-				)
-			)
-		)
-		(property "Footprint" "PCM_JLCPCB:C_0402"
-			(at 102.87 40.64 0)
-			(effects
-				(font
-					(size 1.27 1.27)
-				)
-				(hide yes)
-			)
-		)
-		(property "Datasheet" "~"
-			(at 102.87 40.64 0)
-			(effects
-				(font
-					(size 1.27 1.27)
-				)
-				(hide yes)
-			)
-		)
-		(property "Description" "Unpolarized capacitor, small symbol"
-			(at 102.87 40.64 0)
-			(effects
-				(font
-					(size 1.27 1.27)
-				)
-				(hide yes)
-			)
-		)
-		(pin "2"
-		)
-		(pin "1"
-		)
-		(instances
-			(project "IREC2025_FlightComputer"
-				(path "/d402aac1-6798-4745-a2ce-fc3f8e4c9afb/24d4e930-e2ab-47c0-a5cd-8b7215a2cae3"
-					(reference "C27")
-					(unit 1)
-				)
-			)
-		)
-	)
-	(symbol
 		(lib_id "power:GND")
 		(at 247.65 38.1 0)
@@
 					(unit 1)
 				)
-			)
-		)
-	)
-	(symbol
-		(lib_id "Device:R_Small")
-		(at 110.49 40.64 270)
-		(unit 1)
-		(exclude_from_sim no)
-		(in_bom yes)
-		(on_board yes)
-		(dnp no)
-		(fields_autoplaced yes)
-		(property "Reference" "R11"
-			(at 110.49 35.56 90)
-			(effects
-				(font
-					(size 1.27 1.27)
-				)
-			)
-		)
-		(property "Value" "R"
-			(at 110.49 38.1 90)
-			(effects
-				(font
-					(size 1.27 1.27)
-				)
-			)
-		)
-		(property "Footprint" "Resistor_SMD:R_0402_1005Metric"
-			(at 110.49 40.64 0)
-			(effects
-				(font
-					(size 1.27 1.27)
-				)
-				(hide yes)
-			)
-		)
-		(property "Datasheet" "~"
-			(at 110.49 40.64 0)
-			(effects
-				(font
-					(size 1.27 1.27)
-				)
-				(hide yes)
-			)
-		)
-		(property "Description" "Resistor, small symbol"
-			(at 110.49 40.64 0)
-			(effects
-				(font
-					(size 1.27 1.27)
-				)
-				(hide yes)
-			)
-		)
-		(pin "1"
-		)
-		(pin "2"
-		)
-		(instances
-			(project "IREC2025_FlightComputer"
-				(path "/d402aac1-6798-4745-a2ce-fc3f8e4c9afb/24d4e930-e2ab-47c0-a5cd-8b7215a2cae3"
-					(reference "R11")
-					(unit 1)
-				)

Commit message: update
21/3/2025
Parts:
- removed C28: 10nF, PCM_JLCPCB:C_0402, symbol Device:C_Small
- removed FB2: BLM18AG601SH1D, EasyEDA:L0603, symbol EasyEDA:BLM18AG601SH1D
- removed R9: 10k, Resistor_SMD:R_0402_1005Metric, symbol Device:R_Small
- removed Y1: 32 MHz TCXO, TCXO:OSC_ECS-TXO-2520-33-320-AN-TR, symbol ECS-TXO-2520-33-320-AN-TR:ECS-TXO-2520-33-320-AN-TR
- added C32: 47pF, PCM_JLCPCB:C_0402, symbol PCM_JLCPCB-Capacitors:0402,47pF
- added C34: 1uF, PCM_JLCPCB:C_0402, symbol PCM_JLCPCB-Capacitors:0402,1uF
- added C35: 100nF, PCM_JLCPCB:C_0402, symbol PCM_JLCPCB-Capacitors:0402,100nF
- added L2: BLM18AG121SN1D, EasyEDA:L0603, symbol EasyEDA:BLM18AG121SN1D
- added X2: 1XXD32000MBA, EasyEDA:OSC-SMD_4P-L2.0-W1.6-BL_1XXD, symbol EasyEDA:1XXD32000MBA
- renumbered C35 to C29, C38 to C33, C39 to C36, C33 to C37, C36 to C38, C34 to C39, C37 to C40, C19 to C41, C32 to C42, C26 to C43, C20 to C44, C22 to C45, C23 to C46, C25 to C47, C29 to C48, C24 to C49, C21 to C50, L2 to L4, L4 to L5, L8 to L6, L6 to L7, L7 to L8, L5 to L9, R10 to R18, U4 to U10, U5 to U11
Connections:
- net +3.3V: now also L2.2
- net GND: now also C34.2, C35.2, X2.1 (GND), X2.2 (GND)
- net XTA: now also C32.2
- new net: C34.1, C35.1, L2.1, X2.4 (VCC)
- new net: C32.1, X2.3 (Output)
Other:
- note added: "TCXO_HSE 32MHz"
- note removed: "32MHz TCXO crystal"
- note removed: "600Z @ 100MHz"
- note removed: "Alternatively connect to DIO input for controlling TXCO's output for more power efficiency"
- note removed: "Change to a DIO input for dynamic control over the TCXO functionalities"
- note removed: "Pull up to 3V3 to keep the TCXO output constantly enabled"

Commit message: checkpoint
before the great layout change
Parts:
- removed C29: 3.0pF, PCM_JLCPCB:C_0402, symbol PCM_JLCPCB-Capacitors:0402,3.3pF
- removed C30: 47nF, PCM_JLCPCB:C_0402, symbol PCM_JLCPCB-Capacitors:0402,47pF
- removed C31, C32: 47pF, PCM_JLCPCB:C_0402, symbol PCM_JLCPCB-Capacitors:0402,47pF
- removed C33, C36, C40, C42, C46, C47, C48: C_Small, PCM_JLCPCB:C_0402, symbol Device:C_Small
- removed C34: 1uF, PCM_JLCPCB:C_0402, symbol PCM_JLCPCB-Capacitors:0402,1uF
- removed C35: 100nF, PCM_JLCPCB:C_0402, symbol PCM_JLCPCB-Capacitors:0402,100nF
- removed C44: 1uF, PCM_JLCPCB:C_0402, symbol Device:C_Small
- removed C50: 1nF, PCM_JLCPCB:C_0402, symbol Device:C_Small
- removed JP1: U.FL-R-SMT-1(10), EasyEDA:ANT-SMD_UFL-R-SMT-1-10, symbol EasyEDA:U.FL-R-SMT-1(10)
- removed L3: 47nH, PCM_JLCPCB:C_0402, symbol Device:L_Small
- removed L8: 15nH, Inductor_SMD:L_0603_1608Metric, symbol Device:L_Small
- removed R18: 1k, Resistor_SMD:R_0402_1005Metric, symbol Device:R_Small
- added C27: GJM1555C1H390JB01D, PCM_JLCPCB:C_0402, symbol Device:C_Small
- added C30: 47nF, PCM_JLCPCB:C_0402, symbol Device:C_Small
- added C31, C32: 47pF, PCM_JLCPCB:C_0402, symbol Device:C_Small
- added C34: 1uF, PCM_JLCPCB:C_0402, symbol Device:C_Small
- added C35: 100nF, PCM_JLCPCB:C_0402, symbol Device:C_Small
- added C46, C47: GJM1555C1H3R3BB01D, EasyEDA:C0402, symbol EasyEDA:GJM1555C1H3R3BB01D
- added C48, C50: GRM155R72A102KA01D, EasyEDA:C0402, symbol EasyEDA:GRM155R72A102KA01D
- added C60, C61: 1.8pF, PCM_JLCPCB:C_0402, symbol Device:C_Small
- added L3: 15uH, EasyEDA:L0805, symbol EasyEDA:MLZ2012M150WT000
- added R11: 0R, PCM_JLCPCB:R_0402, symbol EasyEDA:CRCW04020000Z0ED
- added R23, R24: CRCW0402100RFKED, PCM_JLCPCB:R_0402, symbol Device:R_Small
- added RF1: SMA-KE-5, EasyEDA:SMA-TH_SMA-KHDB_C9900020423, symbol EasyEDA:SMA-KE-5
- C37: value C_Small -> 3pF; Name (none) -> GJM1555C1H3R0BB01D
- C38: value C_Small -> 5.6pF; Name (none) -> GJM1555C1H5R6CB01D
- C39: value C_Small -> 2.4pF; Name (none) -> GJM1555C1H2R4BB01D
- C41: value 10nF -> 39pF; Name (none) -> GJM1555C1H390JB01D
- C43: Name (none) -> GRM155R71A474KE01D
- C45: Name (none) -> GRM155R71H104KE14D
- C49: value 10nF -> 1uF; Name (none) -> GRM155R70J105KA12D
- L4: value 0R -> 47nH; footprint Inductor_SMD:L_0402_1005Metric -> PCM_JLCPCB:L_0402; Name (none) -> LQW15AN47NJ00D
- L5: Name (none) -> LQW15AN2N5C00D
- L6: value L_Small -> 4.7nH; Name (none) -> LQW15AN4N7C00D
- L7: value L_Small -> 15nH; Name (none) -> LQW15AN15NH00D
- L9: value L_Small -> LQW15AN9N1H00D; val (none) -> 9.1nH
Connections:
- net +3.3V: no longer C41.2, U10.6 (CTRL#orVDD)
- net ANT_SW: now also R23.1
- net DIO2: now also R24.1
- net GND: now also C30.2, C31.2, C34.2, C35.2, C46.1, C47.1, C48.1, C50.1, C60.2, C61.2, RF1.2, RF1.3, RF1.4, RF1.5; no longer C37.2, C41.1
- net RF1: now also C60.1
- net XTA: now also C32.2
- net at C43.1, U11.7 (VREG): now also L3.1
- net at U10.4 (CTRL): now also C50.2, R24.2
- net at C37.1, L5.1: now also L4.1, R11.2; no longer L4.2
- net at C38.1, L5.2: now also C37.2, C41.1
- net at L7.1, U11.21 (RFI_P): now also C61.1
- net at L6.1: now also C41.2
- net at U10.5 (RFC): now also C27.1
- net at U11.24 (VR_PA): now also L4.2, C30.1, C31.1
- net at U11.23 (RFO): now also R11.1; no longer L4.1
- net at U11.9 (DCC_SW): now also L3.2
- net at L9.2: now also C47.2, RF1.1
- net at L2.1, X2.4 (VCC): now also C34.1, C35.1
- net at X2.3 (Output): now also C32.1
- net at L9.1: now also C27.2, C46.2
- net DIO3 renamed LORA_DIO3
- net LORA_RST renamed LoRa_RST
- new net: C48.2, R23.2, U10.6 (CTRL#orVDD)
Other:
- note added: "DIO1: TXDONE (To GPIO) DIO2: RF Switch DIO3: Interrupt"
- note removed: "Basic Part"
- note removed: "DIO1: TXDONE DIO2: RF Switch DIO3: RXDONE"
- note removed: "Extended Part"
- moved on the sheet: C43, L2, L9

Commit message: 2 designs
Parts:
- renumbered C27 to C?, C30 to C?, C48 to C?, L3 to L?, L2 to L?, R11 to R?, RF1 to RF?
Changed lines of the file:
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@@
 		(on_board yes)
 		(dnp no)
-		(property "Reference" "C27"
+		(property "Reference" "C?"
 			(at 83.82 111.252 90)
 			(effects
@@
 		)
 		(instances
-			(project ""
+			(project "IREC2025_FlightComputer"
 				(path "/d402aac1-6798-4745-a2ce-fc3f8e4c9afb/24d4e930-e2ab-47c0-a5cd-8b7215a2cae3"
-					(reference "C27")
+					(reference "C?")
 					(unit 1)
 				)
@@
 		(on_board yes)
 		(dnp no)
-		(property "Reference" "C30"
+		(property "Reference" "C?"
 			(at 250.19 31.7562 0)
 			(effects
@@
 		)
 		(instances
-			(project ""
+			(project "IREC2025_FlightComputer"
 				(path "/d402aac1-6798-4745-a2ce-fc3f8e4c9afb/24d4e930-e2ab-47c0-a5cd-8b7215a2cae3"
-					(reference "C30")
+					(reference "C?")
 					(unit 1)
 				)
@@
 		(dnp no)
 		(fields_autoplaced yes)
-		(property "Reference" "R11"
+		(property "Reference" "R?"
 			(at 261.62 45.72 0)
 			(effects
@@
 		)
 		(instances
-			(project ""
+			(project "IREC2025_FlightComputer"
 				(path "/d402aac1-6798-4745-a2ce-fc3f8e4c9afb/24d4e930-e2ab-47c0-a5cd-8b7215a2cae3"
-					(reference "R11")
+					(reference "R?")
 					(unit 1)
 				)
@@
 		(on_board yes)
 		(dnp no)
-		(property "Reference" "C48"
+		(property "Reference" "C?"
 			(at 55.88 93.98 0)
 			(effects
@@
 		)
 		(instances
-			(project ""
+			(project "IREC2025_FlightComputer"
 				(path "/d402aac1-6798-4745-a2ce-fc3f8e4c9afb/24d4e930-e2ab-47c0-a5cd-8b7215a2cae3"
-					(reference "C48")
+					(reference "C?")
 					(unit 1)
 				)
@@
 		(dnp no)
 		(fields_autoplaced yes)
-		(property "Reference" "RF1"
+		(property "Reference" "RF?"
 			(at 130.81 132.08 90)
 			(effects
@@
 		)
 		(instances
-			(project ""
+			(project "IREC2025_FlightComputer"
 				(path "/d402aac1-6798-4745-a2ce-fc3f8e4c9afb/24d4e930-e2ab-47c0-a5cd-8b7215a2cae3"
-					(reference "RF1")
+					(reference "RF?")
 					(unit 1)
 				)
@@
 		(on_board yes)
 		(dnp no)
-		(property "Reference" "L3"
+		(property "Reference" "L?"
 			(at 239.014 99.822 90)
 			(effects
@@
 		)
 		(instances
-			(project ""
+			(project "IREC2025_FlightComputer"
 				(path "/d402aac1-6798-4745-a2ce-fc3f8e4c9afb/24d4e930-e2ab-47c0-a5cd-8b7215a2cae3"
-					(reference "L3")
+					(reference "L?")
 					(unit 1)
 				)
@@
 		(on_board yes)
 		(dnp no)
-		(property "Reference" "L2"
+		(property "Reference" "L?"
 			(at 54.864 34.798 0)
 			(effects
@@
 		)
 		(instances
-			(project ""
+			(project "IREC2025_FlightComputer"
 				(path "/d402aac1-6798-4745-a2ce-fc3f8e4c9afb/24d4e930-e2ab-47c0-a5cd-8b7215a2cae3"
-					(reference "L2")
+					(reference "L?")
 					(unit 1)
 				)

Commit message: changed most resistors to 0603
Parts:
- removed C31, C32: 47pF, PCM_JLCPCB:C_0402, symbol Device:C_Small
- removed C34, C49: 1uF, PCM_JLCPCB:C_0402, symbol Device:C_Small
- removed C35, C45: 100nF, PCM_JLCPCB:C_0402, symbol Device:C_Small
- removed C37: 3pF, PCM_JLCPCB:C_0402, symbol Device:C_Small
- removed C38: 5.6pF, PCM_JLCPCB:C_0402, symbol Device:C_Small
- removed C39: 2.4pF, PCM_JLCPCB:C_0402, symbol Device:C_Small
- removed C41: 39pF, PCM_JLCPCB:C_0402, symbol Device:C_Small
- removed C43: 470nF, PCM_JLCPCB:C_0402, symbol Device:C_Small
- removed C46, C47: GJM1555C1H3R3BB01D, EasyEDA:C0402, symbol EasyEDA:GJM1555C1H3R3BB01D
- removed C50, C?: GRM155R72A102KA01D, EasyEDA:C0402, symbol EasyEDA:GRM155R72A102KA01D
- removed C60, C61: 1.8pF, PCM_JLCPCB:C_0402, symbol Device:C_Small
- removed C?: GJM1555C1H390JB01D, PCM_JLCPCB:C_0402, symbol Device:C_Small
- removed C?: 47nF, PCM_JLCPCB:C_0402, symbol Device:C_Small
- removed L4: 47nH, PCM_JLCPCB:L_0402, symbol Device:L_Small
- removed L5: 2.5nH, PCM_JLCPCB:C_0402, symbol Device:L_Small
- removed L6: 4.7nH, Inductor_SMD:L_0402_1005Metric, symbol Device:L_Small
- removed L7: 15nH, Inductor_SMD:L_0402_1005Metric, symbol Device:L_Small
- removed L9: LQW15AN9N1H00D, Inductor_SMD:L_0402_1005Metric, symbol Device:L_Small
- removed L?: 15uH, EasyEDA:L0805, symbol EasyEDA:MLZ2012M150WT000
- removed L?: BLM18AG121SN1D, EasyEDA:L0603, symbol EasyEDA:BLM18AG121SN1D
- removed R23, R24: CRCW0402100RFKED, PCM_JLCPCB:R_0402, symbol Device:R_Small
- removed R?: 0R, PCM_JLCPCB:R_0402, symbol EasyEDA:CRCW04020000Z0ED
- removed U10: PE4259-63, EasyEDA:SC-70-6_L2.2-W1.3-P0.65-LS2.1-BL, symbol EasyEDA:PE4259-63
- removed U11: SX1262IMLTRT, Package_DFN_QFN:QFN-24-1EP_4x4mm_P0.5mm_EP2.6x2.6mm, symbol RF:SX1262IMLTRT
- removed X2: 1XXD32000MBA, EasyEDA:OSC-SMD_4P-L2.0-W1.6-BL_1XXD, symbol EasyEDA:1XXD32000MBA
- added C27: 100nF, PCM_JLCPCB:C_0402, symbol Device:C_Small
- added C34: 10uF, PCM_JLCPCB:C_0402, symbol PCM_JLCPCB-Capacitors:0402,10uF
- added U15: ~, LORAMODF:G-NiceRF LoRa1262-915, symbol LoRaMod:G-NiceRF_LoRa1262-915
- gave numbers to parts that had none: 1
Connections:
- net +3.3V: now also C27.1, C34.1, U15.13 (VCC)
- net BUSY: now also U15.16 (BUSY)
- net DIO1: now also U15.15 (DIO1)
- net GND: now also C27.2, C34.2, U15.1 (GND), U15.10 (GND), U15.8 (GND)
- net LORA_DIO3: now also U15.11 (DIO3)
- net LoRa_MISO: now also U15.2 (MISO)
- net LoRa_MOSI: now also U15.3 (MOSI)
- net LoRa_NSS: now also U15.5 (NSS)
- net LoRa_RST: now also U15.6 (NRESET)
- net LoRa_SCLK: now also U15.4 (SCK)
- net at RF1.1: now also U15.9 (ANT)
- no-connect marks 1 -> 0
Other:
- note added: "CL21B106KOQNNNE"
- note removed: "From GPIO"
- note removed: "PE4259 Switch"
- note removed: "SX1262 + Matching"
- note removed: "TCXO_HSE 32MHz"
- moved on the sheet: RF1
