File: IREC2025_FlightComputer.kicad_pcb (KiCad board)
At the start: 4 copper layers, 63.5 x 99 mm, 120 parts, among them J1 Molex Microfit, J2 BOOT0, J3 Companion, J5 SWD, Q1 SI7232DN-T1-GE3, U1 STM32U575VGTx, U12 ADXL375BCCZ-RL7, U14 SAM-M10Q-00B, U2 MMC5983MA, U3 BMI088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

Commit message: Special version
Parts:
- added R23: 5R, pyrolim:RES_3540_TEC, B.Cu at (80.8, 137.3)
- added R25: 5R, pyrolim:RES_3540_TEC, B.Cu at (74.2, 137.3)
- moved J1 9.97 mm to (102.0, 145.8)
- moved Pyro_CH1 7.59 mm to (81.5, 145.8)
- moved Pyro_CH2 7.54 mm to (70.0, 145.8)
- moved H1 6.25 mm to (118.8, 146.4)
- moved H2 6.25 mm to (62.2, 146.4)
Connections:
- Pyro_CH1 pad 2: VBAT+ -> Net-(Pyro_CH1-Pin_2)
- Pyro_CH2 pad 2: VBAT+ -> Net-(Pyro_CH2-Pin_2)
- Q1 pad 5: Net-(Pyro_CH2-Pin_1) -> Net-(Pyro_CH1-Pin_1)
- Q1 pad 6: Net-(Pyro_CH2-Pin_1) -> Net-(Pyro_CH1-Pin_1)
- Q1 pad 7: Net-(Pyro_CH1-Pin_1) -> Net-(Pyro_CH2-Pin_1)
- Q1 pad 8: Net-(Pyro_CH1-Pin_1) -> Net-(Pyro_CH2-Pin_1)
Routing:
- net VBAT+: track 23.6 -> 0.00 mm
- net Net-(Pyro_CH1-Pin_1): track 13.0 -> 34.5 mm
- net Net-(Pyro_CH2-Pin_1): track 10.4 -> 18.4 mm
- added copper zone on F.Cu, net Net-(Pyro_CH1-Pin_2)
- added copper zone on F.Cu, net Net-(Pyro_CH2-Pin_2)
Other:
- board size 63.5 x 99 mm -> 63.5 x 105.3 mm
- board text added: "By Thanapat Suwanrat Boonyakorn Tanrattanakorn"
- board text added: "CURSR-IV Flight Computer"
- board text removed: "CURSR-IV Flight Computer By Thanapat Suwanrat Boonyakorn Tanrattanakorn"

Commit message: v2 manufactured ver.
Parts:
- moved J1 10.6 mm to (108.5, 137.4)
- moved Pyro_CH2 6.44 mm to (69.3, 139.4)
- moved Pyro_CH1 6.25 mm to (81.3, 139.6)
- moved H1 6.25 mm to (118.8, 140.1)
- moved H2 6.25 mm to (62.2, 140.1)
- moved R25 5.66 mm to (72.4, 132.0)
- moved R23 5.51 mm to (78.6, 132.2)
Connections:
- Q1 pad 5: Net-(Pyro_CH1-Pin_1) -> Net-(Pyro_CH2-Pin_1)
- Q1 pad 6: Net-(Pyro_CH1-Pin_1) -> Net-(Pyro_CH2-Pin_1)
- Q1 pad 7: Net-(Pyro_CH2-Pin_1) -> Net-(Pyro_CH1-Pin_1)
- Q1 pad 8: Net-(Pyro_CH2-Pin_1) -> Net-(Pyro_CH1-Pin_1)
Routing:
- net Net-(Pyro_CH1-Pin_1): track 34.5 -> 13.2 mm
- net Net-(Pyro_CH1-Pin_2): track 0.00 -> 14.7 mm
- net Net-(Pyro_CH2-Pin_1): track 18.4 -> 11.8 mm
- net Net-(Pyro_CH2-Pin_2): track 0.00 -> 4.68 mm
- net VBAT-: track 96.9 -> 97.3 mm, vias 207 -> 191
- net VBAT+: vias 0 -> 1
- added copper zone on B.Cu, net VBAT+
- removed copper zone on F.Cu, net Net-(Pyro_CH1-Pin_2)
- removed copper zone on F.Cu, net Net-(Pyro_CH2-Pin_2)
Other:
- board size 63.5 x 105.3 mm -> 63.5 x 99 mm

Commit message: Final manu v2
Parts:
- R24: footprint PCM_JLCPCB:R_0805 -> pyrolim:RES_3540_TEC; moved to B.Cu
- moved R24 2.35 mm to (68.1, 127.8), turned to -90 degrees
- moved R25 1.08 mm to (73.5, 132.2)
- moved SERVO1 0.47 mm to (62.7, 108.5)
- moved SERVO2 0.47 mm to (62.7, 123.5)
Routing:
- net Net-(SERVO1-Pin_2): track 22.0 -> 24.2 mm
- net +5V: track 48.7 -> 49.3 mm
- net VBAT-: vias 191 -> 182
