File: IREC2025_FlightComputer.kicad_pcb (KiCad board)
At the start: 4 copper layers, 63.5 x 99 mm, 122 parts, among them J1 Molex Microfit, J2 BOOT0, J3 Companion, J5 SWD, Q1 SI7232DN-T1-GE3, U1 STM32U575VGTx, U12 ADXL375BCCZ-RL7, U14 SAM-M10Q-00B, U2 MMC5983MA, U3 BMI088, U4 TMP275AIDGKR VSSOP8, U5 LP5912Q3.3DRVRQ1, U6 MS5607-02BA, U7 THGBMUG6C1LBAIL, U8 TPS62153, U9 SN74HCT125DR, X1 1XXD32000MBA

Commit message: Complete Redesign
Parts:
- removed the G*** at (82.6, 66.0)
- removed the G*** at (95.5, 108.1)
- removed the G*** at (99.7, 61.4)
- removed LOGO (x2): LOGO, Cuharlogo:CUHARLOGOMOD
- added C19: 1uF, PCM_JLCPCB:C_0603, F.Cu at (153.0, 236.5)
- added C2: 220UF 16V, EasyEDA:CAP-SMD_BD6.3-L6.6-W6.6-LS7.4-FD, F.Cu at (162.5, 237.0)
- added C29: 100nF, PCM_JLCPCB:C_0603, F.Cu at (157.2, 235.2)
- added C3: 470uF, Capacitor_SMD:CP_Elec_8x10, F.Cu at (117.2, 234.5)
- added C31: 100nF, PCM_JLCPCB:C_0603, F.Cu at (126.0, 237.0)
- added D7: SS34_C466502, GNSS:DIOM7959X262N, F.Cu at (132.2, 221.0)
- added G***: LOGO, LOGO, F.Cu at (165.0, 75.0)
- added J4: Molex Microfit, Connector_Molex:Molex_Micro-Fit_3.0_43650-0215_1x02_P3.00mm_Vertical, F.Cu at (104.5, 234.8)
- added J6: Molex Microfit, Connector_Molex:Molex_Micro-Fit_3.0_43650-0215_1x02_P3.00mm_Vertical, F.Cu at (172.5, 237.5)
- added J7: U.FL, PCM_JLCPCB:IPEX-SMD_BWIPX-1-001E, F.Cu at (167.2, 131.5)
- added J8: MEM2080-00-128-00-A_REVA, SDCard:GCT_MEM2080-00-128-00-A_REVA, F.Cu at (186.5, 88.6)
- added L2: 33uH,5A, Inductor_SMD:L_Bourns_SRR1208_12.7x12.7mm, F.Cu at (135.7, 231.8)
- added R26: 10kΩ, PCM_JLCPCB:R_0603, F.Cu at (75.0, 162.3)
- added R27: 10kΩ, PCM_JLCPCB:R_0603, F.Cu at (75.0, 164.5)
- added R28: 10kΩ, PCM_JLCPCB:R_0603, F.Cu at (75.0, 166.8)
- added R29: 10kΩ, PCM_JLCPCB:R_0603, F.Cu at (75.0, 169.0)
- added R30: 10kΩ, PCM_JLCPCB:R_0603, F.Cu at (78.6, 157.8)
- added R31: 1MΩ, PCM_JLCPCB:R_0603, F.Cu at (195.1, 88.7)
- added R31: 10kΩ, PCM_JLCPCB:R_0603, F.Cu at (78.6, 160.0)
- added R32: 10kΩ, PCM_JLCPCB:R_0603, F.Cu at (78.6, 162.3)
- added R33: 10kΩ, PCM_JLCPCB:R_0603, F.Cu at (78.6, 164.5)
- added R35: 10kΩ, PCM_JLCPCB:R_0603, F.Cu at (78.6, 166.1)
- added R8: 10kΩ, PCM_JLCPCB:R_0603, F.Cu at (148.0, 238.4)
- added U10: XL4015E1, EasyEDA:TO-263-5_L10.2-W8.9-P1.70-TL, F.Cu at (150.5, 228.5)
- added U11: XTSD08GLGEAG, EasyEDA:LGA-8_L6.0-W8.0-P1.27-BL, B.Cu at (186.1, 81.6)
- C1, C10, C11, C12, C13, C18, C30, C33, C36, C4, C40, C42, C44, C48, C5, C53, C58, C6, C7, C8, C9, R11, R12, R13, R14, R15, R19, R21, R3, R34, R4, R6, R7, X1: moved to B.Cu
- R23, R25: value 5R -> 10kΩ; footprint pyrolim:RES_3540_TEC -> PCM_JLCPCB:R_0603; moved to F.Cu
- R24: value 8.87R -> 3.3kΩ; footprint pyrolim:RES_3540_TEC -> PCM_JLCPCB:R_0603; moved to F.Cu
- moved U7 412.1 mm to (392.7, 342.5)
- moved R57 405.7 mm to (367.1, 349.8), turned to 0 degrees
- moved C73 402.5 mm to (370.9, 343.1), turned to 0 degrees
- moved R58 392.0 mm to (367.1, 352.1)
- moved R56 385.3 mm to (367.1, 347.6)
- moved R52 384.1 mm to (363.5, 352.1), turned to 0 degrees
- moved R53 384.0 mm to (363.5, 354.3), turned to 0 degrees
- moved R55 382.9 mm to (367.1, 345.3), turned to 0 degrees
- moved R54 378.3 mm to (367.1, 343.1), turned to 0 degrees
- moved R49 377.8 mm to (363.5, 345.3), turned to 0 degrees
- moved R50 377.5 mm to (363.5, 347.6), turned to 0 degrees
- moved R51 377.1 mm to (363.5, 349.8), turned to 0 degrees
- moved H1 263.3 mm to (-110.5, 10.5), turned to 0 degrees
- moved H3 230.4 mm to (-110.5, 24.8), turned to 0 degrees
- moved J3 220.2 mm to (-92.9, 43.4), turned to 0 degrees
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Connections:
- D3 pad 2: Net-(J1-Pin_1) -> Net-(J1-Pin_2)
- J1 pad 1: Net-(J1-Pin_1) -> VBAT-
- J1 pad 2: VBAT- -> Net-(J1-Pin_2)
- Pyro_CH1 pad 1: Net-(Pyro_CH1-Pin_1) -> VBAT+
- Pyro_CH2 pad 2: Net-(Pyro_CH2-Pin_2) -> VBAT+
- Q1 pad 7: Net-(Pyro_CH1-Pin_1) -> Net-(Pyro_CH1-Pin_2)
- Q1 pad 8: Net-(Pyro_CH1-Pin_1) -> Net-(Pyro_CH1-Pin_2)
- R23 pad 1: VBAT+ -> +3.3V
- R23 pad 2: Net-(Pyro_CH1-Pin_2) -> DAT0
- R24 pad 1: +5V -> Net-(U10-FB)
- R24 pad 2: Net-(SERVO1-Pin_2) -> VBAT-
- R25 pad 1: VBAT+ -> +3.3V
- R25 pad 2: Net-(Pyro_CH2-Pin_2) -> DAT1
- RF1 pad 1: Net-(U15-ANT) -> unconnected-(RF1-Pad1)
- RF1 pad 2: VBAT- -> unconnected-(RF1-Pad2)
- RF1 pad 3: VBAT- -> unconnected-(RF1-Pad3)
- RF1 pad 4: VBAT- -> unconnected-(RF1-Pad4)
- RF1 pad 5: VBAT- -> unconnected-(RF1-Pad5)
- SERVO1 pad 2: Net-(SERVO1-Pin_2) -> +5Vservo
- SERVO2 pad 2: Net-(SERVO1-Pin_2) -> +5Vservo
- U1 pad 15: unconnected-(U1-PC0-Pad15) -> BAT_LEVEL
- U1 pad 16: eMMC_CLK -> unconnected-(U1-PC1-Pad16)
- U1 pad 17: ADXL_MISO -> unconnected-(U1-PC2-Pad17)
- U1 pad 18: ADXL_MOSI -> MS5607_MOSI
- U1 pad 36: unconnected-(U1-PB1-Pad36) -> LoRa_RST
- U1 pad 41: ADXL_INT2 -> unconnected-(U1-PE10-Pad41)
- U1 pad 42: ADXL_INT1 -> unconnected-(U1-PE11-Pad42)
- U1 pad 43: LoRa_RST -> unconnected-(U1-PE12-Pad43)
- U1 pad 47: ADXL_SCLK -> unconnected-(U1-PB10-Pad47)
- U1 pad 51: ADXL_NSS -> unconnected-(U1-PB12-Pad51)
- U1 pad 53: DAT0 -> unconnected-(U1-PB14-Pad53)
- U1 pad 54: DAT1 -> unconnected-(U1-PB15-Pad54)
- U1 pad 58: RST_n -> unconnected-(U1-PD11-Pad58)
- U1 pad 63: DAT6 -> unconnected-(U1-PC6-Pad63)
- U1 pad 64: DAT7 -> unconnected-(U1-PC7-Pad64)
- U1 pad 65: unconnected-(U1-PC8-Pad65) -> BMI_GYRO_INT2
- U1 pad 66: unconnected-(U1-PC9-Pad66) -> BMI_GYRO_INT1
- U1 pad 67: unconnected-(U1-PA8-Pad67) -> MS5607_CS
- U1 pad 68: unconnected-(U1-PA9-Pad68) -> MS5607_SCLK
- U1 pad 77: MS5607_NSS -> unconnected-(U1-PA15-Pad77)
- U1 pad 78: BMI_SCLK -> ADXL_SCLK
- U1 pad 79: BMI_MISO -> ADXL_MISO
- U1 pad 80: BMI_MOSI -> ADXL_MOSI
- U1 pad 81: BMI_GYRO_CS -> BMI_accel_INT1
- U1 pad 82: unconnected-(U1-PD1-Pad82) -> BMI_accel_INT2
- U1 pad 83: BMI_GYRO_INT1 -> BMI_GYRO_CS
- U1 pad 84: BMI_GYRO_INT2 -> MS5607_MISO
- U1 pad 85: BMI_accel_CS -> ADXL_INT2
- U1 pad 86: BMI_accel_INT1 -> ADXL_INT1
- U1 pad 87: BMI_accel_INT2 -> BMI_accel_CS
- U1 pad 88: eMMC_CMD -> unconnected-(U1-PD7-Pad88)
- U1 pad 89: DAT2 -> unconnected-(U1-PB3-Pad89)
- U1 pad 90: DAT3 -> unconnected-(U1-PB4-Pad90)
- U1 pad 95: DAT4 -> unconnected-(U1-PB8-Pad95)
- U1 pad 96: DAT5 -> unconnected-(U1-PB9-Pad96)
- U1 pad 97: BAT_LEVEL -> ADXL_CS
- U12 pad 7: ADXL_NSS -> ADXL_CS
- U15 pad 9: Net-(U15-ANT) -> Net-(J7-In)
- U3 pad 10: BMI_MISO -> ADXL_MISO
- U3 pad 15: BMI_MISO -> ADXL_MISO
- U3 pad 8: BMI_SCLK -> ADXL_SCLK
- U3 pad 9: BMI_MOSI -> ADXL_MOSI
- U6 pad 4: MS5607_NSS -> MS5607_CS
- U6 pad 5: MS5607_NSS -> MS5607_CS
- U6 pad 6: BMI_MISO -> MS5607_MISO
- U6 pad 7: BMI_MOSI -> MS5607_MOSI
- U6 pad 8: BMI_SCLK -> MS5607_SCLK
Routing:
- net VBAT-: track 97.3 -> 0.00 mm, vias 182 -> 0
- net Net-(U14-TXD): track 7.02 -> 92.1 mm, vias 2 -> 1
- net Net-(U14-RXD): track 6.88 -> 90.2 mm, vias 2 -> 1
- net +3.3V: track 114.7 -> 43.8 mm, vias 30 -> 14
- net GNSS_INT: track 46.5 -> 115.2 mm
- net GNSS_RST: track 44.9 -> 111.2 mm, vias 2 -> 4
- net Backup: track 58.2 -> 0.00 mm, vias 2 -> 0
- net DAT5: track 54.1 -> 0.00 mm, vias 2 -> 0
- net eMMC_CLK: track 58.5 -> 6.08 mm, vias 3 -> 1
- net DAT4: track 49.5 -> 0.00 mm, vias 2 -> 0
- net +5V: track 49.3 -> 0.00 mm, vias 3 -> 0
- net eMMC_CMD: track 49.6 -> 3.37 mm, vias 2 -> 1
- net LoRa_MOSI: track 63.6 -> 18.2 mm, vias 0 -> 2
- net DAT3: track 47.2 -> 5.45 mm, vias 4 -> 1
- net GNSS_SAFEBOOT: track 41.1 -> 0.00 mm, vias 2 -> 0
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- added copper zone on F.Cu, net Net-(D7-Pad2)
- removed copper zone on In2.Cu, net +3.3V
- removed copper zone on F.Cu, net +3.3VA
- removed copper zone on F.Cu, net +5V
- removed copper zone on F.Cu, net Net-(D4-K)
- removed copper zone on F.Cu, net Net-(J1-Pin_1)
- removed copper zone on F.Cu, net Net-(L1-Pad1)
- removed copper zone on B.Cu, net VBAT+
- removed copper zone on F.Cu, net VBAT+
- removed copper zone on B.Cu, net VBAT-
- removed copper zone on F.Cu, net VBAT-
- removed copper zone on In1.Cu, net VBAT-
- removed copper zone on F.Cu, net VBUS
Other:
- board size 63.5 x 99 mm -> 165.2 x 176 mm
- board text removed: "0"
- board text removed: "1"
- board text removed: "3V3"
- board text removed: "BOOT0"
- board text removed: "BUSY"
- board text removed: "Battery"
- board text removed: "By Thanapat Suwanrat Boonyakorn Tanrattanakorn"
- board text removed: "C11"
- board text removed: "C17"
- board text removed: "C18"
- board text removed: "C20"
- board text removed: "C24"
- board text removed: "C28"
- board text removed: "C4"
- board text removed: "C7"
- board text removed: "C70"
- board text removed: "C74"
- board text removed: "COMPANION RX"
- board text removed: "COMPANION TX"
- board text removed: "CURSR-IV Flight Computer"
- board text removed: "D1"
- board text removed: "D4"
- board text removed: "D5"
- board text removed: "D6"
- board text removed: "GND"
- board text removed: "GNSS"
- board text removed: "L1"
- board text removed: "PWR"
- board text removed: "PYRO1"
- board text removed: "PYRO2"
- board text removed: "R12"
- board text removed: "R15"
- board text removed: "R16"
- board text removed: "R17"
- board text removed: "R2"
- board text removed: "R3"
- board text removed: "SI7232DN"
- board text removed: "SWCLK"
- board text removed: "SWDIO"
- board text removed: "U5"
- board text removed: "U8"
- board text removed: "U9"
- board text removed: "eMMC"

Commit message: 1
Parts:
- removed C73: 10uF, PCM_JLCPCB:C_0603
- removed J7: U.FL, PCM_JLCPCB:IPEX-SMD_BWIPX-1-001E
- removed the R31 at (78.6, 160.0)
- removed R49, R50, R51, R52, R53, R54, R55, R56, R57: 22kΩ, PCM_JLCPCB:R_0603
- removed R58: 47kΩ, PCM_JLCPCB:R_0603
- removed U7: THGBMUG6C1LBAIL, EasyEDA:BGA-153_L13.0-W11.5-P0.50-TL_KLM8G1GEME-B041
- added C32: 100nF, PCM_JLCPCB:C_0603, B.Cu at (127.8, 119.0)
- R16, R17, R23, R25, R26, R27, R31, R35: moved to B.Cu
- moved H1 280.4 mm to (143.3, 129.8)
- moved H4 280.1 mm to (166.8, 72.2)
- moved RF1 205.0 mm to (165.5, 129.8)
- moved R28 204.4 mm to (277.8, 140.8)
- moved R29 204.4 mm to (277.8, 143.0)
- moved R30 199.5 mm to (277.8, 145.2)
- moved R33 184.4 mm to (261.9, 144.8)
- moved R16 177.8 mm to (95.5, 99.2), turned to -90 degrees
- moved R17 176.3 mm to (95.5, 96.0), turned to 90 degrees
- moved R32 175.4 mm to (253.2, 144.8)
- moved H3 170.4 mm to (23.2, 130.5)
- moved H2 144.4 mm to (23.2, 72.2)
- moved R5 125.6 mm to (96.4, 129.8)
- moved LS1 122.8 mm to (104.1, 124.3), turned to -45 degrees
- moved BT1 109.0 mm to (42.4, 74.8)
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Connections:
- J8 pad P4: unconnected-(J8-VDD-PadP4) -> +3.3V
- RF1 pad 1: unconnected-(RF1-Pad1) -> Net-(U15-ANT)
- RF1 pad 2: unconnected-(RF1-Pad2) -> VBAT-
- RF1 pad 3: unconnected-(RF1-Pad3) -> VBAT-
- RF1 pad 4: unconnected-(RF1-Pad4) -> VBAT-
- RF1 pad 5: unconnected-(RF1-Pad5) -> VBAT-
- U1 pad 16: unconnected-(U1-PC1-Pad16) -> eMMC_CLK
- U1 pad 53: unconnected-(U1-PB14-Pad53) -> DAT0
- U1 pad 54: unconnected-(U1-PB15-Pad54) -> DAT1
- U1 pad 88: unconnected-(U1-PD7-Pad88) -> eMMC_CMD
- U1 pad 89: unconnected-(U1-PB3-Pad89) -> DAT2
- U1 pad 90: unconnected-(U1-PB4-Pad90) -> DAT3
- U15 pad 9: Net-(J7-In) -> Net-(U15-ANT)
Routing:
- net Net-(U14-TXD): track 92.1 -> 19.8 mm
- net GNSS_TX: track 14.1 -> 81.2 mm
- net DAT0: track 5.74 -> 56.3 mm, vias 1 -> 3
- net DAT3: track 5.45 -> 54.4 mm, vias 1 -> 6
- net SERVO_B: track 0.00 -> 48.2 mm, vias 0 -> 2
- net DAT1: track 8.73 -> 55.9 mm, vias 1 -> 5
- net DAT2: track 5.37 -> 50.7 mm, vias 1 -> 5
- net eMMC_CMD: track 3.37 -> 42.7 mm, vias 1 -> 6
- net Backup: track 0.00 -> 37.6 mm, vias 0 -> 2
- net SERVO_A: track 0.00 -> 26.9 mm
- net eMMC_CLK: track 6.08 -> 27.9 mm, vias 1 -> 2
- net LoRa_MISO: track 16.2 -> 8.43 mm
- net BUSY: track 28.5 -> 20.7 mm
- net Net-(U14-RXD): track 90.2 -> 82.7 mm
- net LoRa_MOSI: track 18.2 -> 11.2 mm
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- added copper zone on In2.Cu, net +3.3V
- added copper zone on B.Cu, net VBAT-
- added copper zone on F.Cu, net VBAT-
- added copper zone on In1.Cu, net VBAT-

Commit message: Update IREC2025_FlightComputer.kicad_pcb
Parts:
- moved D5 55.2 mm to (99.5, 86.6)
- moved D4 53.2 mm to (91.7, 86.6)
- moved C23 39.5 mm to (90.7, 83.6), turned to 180 degrees
- moved R10 27.3 mm to (84.8, 75.5)
- moved C24 14.9 mm to (76.7, 84.6), turned to 180 degrees
- moved C70 14.6 mm to (76.8, 86.6), turned to 180 degrees
- moved G*** 8.49 mm to (167.0, 78.2)
- moved C20 0.48 mm to (81.8, 83.8)
- moved D3 0.48 mm to (74.0, 79.9)
- moved J1 0.48 mm to (75.9, 73.0)
- moved L1 0.48 mm to (88.8, 79.8)
- moved R1 0.48 mm to (89.5, 71.5)
- moved U8 0.48 mm to (83.2, 79.9)
Routing:
- net +5V: track 0.00 -> 1.68 mm
- added copper zone on F.Cu, net +5V
- added copper zone on F.Cu, net Net-(L1-Pad1)

Commit message: updated SD
Parts:
- C32, U11: moved to F.Cu
- J8: moved to B.Cu
- moved C32 52.9 mm to (83.8, 148.4), turned to 90 degrees
- moved R31 19.2 mm to (133.3, 115.8), turned to 0 degrees
- moved U11 13.3 mm to (119.2, 124.8)
- moved R27 12.2 mm to (139.1, 115.0)
- moved R35 11.3 mm to (141.9, 128.4), turned to 135 degrees
- moved J8 7.33 mm to (132.6, 125.9), turned to 0 degrees
- moved H1 6.19 mm to (149.5, 129.8)
- moved R26 6.13 mm to (141.7, 124.7)
- moved R23 5.09 mm to (144.7, 127.4)
- moved R25 3.44 mm to (146.4, 124.7)
Routing:
- net eMMC_CLK: track 27.9 -> 54.9 mm, vias 2 -> 3
- net eMMC_CMD: track 42.7 -> 18.2 mm, vias 6 -> 2
- net DAT2: track 50.7 -> 72.2 mm, vias 5 -> 6
- net DAT3: track 54.4 -> 71.8 mm
- net DAT0: track 56.3 -> 69.5 mm
- net DAT1: track 55.9 -> 62.8 mm
- net +3.3V: track 47.2 -> 43.9 mm, vias 16 -> 14
- net Net-(J8-SHIELD): vias 1 -> 0
- removed copper zone on In2.Cu, net +3.3V

Commit message: .
Parts:
- added C35: 180uF, 180uF:CAP_FKS_F_PAN, F.Cu at (21.7, 187.5)
- added C37: 1uF, PCM_JLCPCB:C_0603, F.Cu at (42.7, 166.7)
- added C38: 470uF, Capacitor_SMD:CP_Elec_8x10, F.Cu at (34.1, 187.3)
- added D8: SS34_C466502, GNSS:DIOM7959X262N, F.Cu at (45.2, 186.3)
- added L3: 68uH, EasyEDA:IND-SMD_L22.5-W22.0, F.Cu at (27.8, 170.8)
- added U7: XL1509-5.0, Package_SO:SOIC-8_3.9x4.9mm_P1.27mm, F.Cu at (45.0, 162.3)
- moved R5 0.89 mm to (97.3, 129.8), turned to 180 degrees
- moved LS1 0.58 mm to (104.0, 123.8)

Commit message: ..
Parts:
- C16, C22, C26, C28, FB1, R38, R9: moved to B.Cu
- moved J3 267.8 mm to (168.0, 103.8), turned to 180 degrees
- moved R38 266.5 mm to (185.4, 113.6), turned to 45 degrees
- moved C22 265.1 mm to (183.9, 112.1), turned to -135 degrees
- moved J5 243.2 mm to (153.3, 71.4), turned to -90 degrees
- moved FB1 227.7 mm to (127.9, 109.2), turned to 180 degrees
- moved C26 225.1 mm to (148.3, 101.3)
- moved C14 217.6 mm to (131.6, 107.2), turned to 135 degrees
- moved C15 217.3 mm to (130.5, 108.2), turned to 135 degrees
- moved C16 211.6 mm to (125.2, 108.4), turned to 90 degrees
- moved J2 203.0 mm to (117.5, 71.3), turned to -90 degrees
- moved R9 195.4 mm to (115.0, 75.0), turned to -90 degrees
- moved C28 181.2 mm to (103.5, 101.8)
- moved R39 51.5 mm to (-24.2, 65.2), turned to 180 degrees
- moved LED3 45.5 mm to (-24.3, 61.5)
- moved PB0 42.8 mm to (-107.6, 34.8)
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Connections:
- U1 pad 13: unconnected-(U1-PH1-Pad13) -> GNSS_SAFEBOOT
- U1 pad 44: GNSS_SAFEBOOT -> unconnected-(U1-PE13-Pad44)
Routing:
- net GNSS_SAFEBOOT: track 0.00 -> 99.8 mm, vias 0 -> 4
- net COMPANION_RX: track 0.00 -> 30.8 mm, vias 0 -> 1
- net COMPANION_TX: track 0.00 -> 30.8 mm, vias 0 -> 1
- net Net-(U1-PH3): track 0.00 -> 24.7 mm, vias 0 -> 2
- net SWDIO: track 0.00 -> 23.1 mm
- net SWCLK: track 0.00 -> 22.8 mm, vias 0 -> 2
- net Net-(U14-RXD): track 82.7 -> 74.2 mm
- net GNSS_TX: track 81.2 -> 75.1 mm
- net GNSS_INT: track 115.4 -> 109.3 mm
- net GNSS_RST: track 111.2 -> 105.9 mm
- net BOOT0: track 0.00 -> 2.93 mm, vias 0 -> 1
- net Net-(U1-VCAP): track 0.00 -> 2.60 mm, vias 0 -> 1
- net GNSS_RX: track 17.6 -> 20.2 mm
- net USB_DN: track 54.9 -> 52.5 mm
- net +3.3V: track 43.9 -> 45.9 mm
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- added copper zone on F.Cu, net +3.3VA
Other:
- board text added: "3v3"
- board text added: "BOOT0"
- board text added: "CLK"
- board text added: "DIO"
- board text added: "Debug"
- board text added: "GND"
- board text added: "UART"
