File: IREC2025_FlightComputer.kicad_sch (KiCad schematic)
At the start: 72 parts, among them J1 Molex Microfit, J2 BOOT0, J3 Companion, J5 SWD, Q1 SI7232DN-T1-GE3, U1 STM32U575VGTx, U5 LP5912Q3.3DRVRQ1, U8 TPS62153, U9 SN74HCT125DR, X1 1XXD32000MBA

Commit message: Final manu v2
Parts:
- R24: footprint PCM_JLCPCB:R_0805 -> pyrolim:RES_3540_TEC
Changed lines of the file:
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@@
 			)
 		)
-		(property "Footprint" "PCM_JLCPCB:R_0805"
+		(property "Footprint" "pyrolim:RES_3540_TEC"
 			(at 313.182 186.69 90)
 			(effects

Commit message: Complete Redesign
Parts:
- removed R23, R25: 5R, pyrolim:RES_3540_TEC, symbol PCM_JLCPCB-Resistors:0402,470Ω
- removed R24: 8.87R, pyrolim:RES_3540_TEC, symbol PCM_JLCPCB-Resistors:0603,1kΩ
- added C19: 1uF, PCM_JLCPCB:C_0603, symbol PCM_JLCPCB-Capacitors:0402,1uF
- added C2: 220UF 16V, EasyEDA:CAP-SMD_BD6.3-L6.6-W6.6-LS7.4-FD, symbol EasyEDA:220UF16V铝电解电容
- added C29, C31: 100nF, PCM_JLCPCB:C_0603, symbol PCM_JLCPCB-Capacitors:0402,100nF
- added C3: 470uF, Capacitor_SMD:CP_Elec_8x10, symbol PCM_JLCPCB-Capacitors:Plugin,D10xL16mm,470uF
- added D7: SS34_C466502, GNSS:DIOM7959X262N, symbol EasyEDA:SS34_C466502
- added J4, J6: Molex Microfit, Connector_Molex:Molex_Micro-Fit_3.0_43650-0215_1x02_P3.00mm_Vertical, symbol Connector:Conn_01x02_Socket
- added L2: 33uH,5A, Inductor_SMD:L_Bourns_SRR1208_12.7x12.7mm, symbol 33uHcoil:2107-H-RC
- added R24: 3.3kΩ, PCM_JLCPCB:R_0603, symbol PCM_JLCPCB-Resistors:0603,3.3kΩ
- added R8: 10kΩ, PCM_JLCPCB:R_0603, symbol PCM_JLCPCB-Resistors:0603,10kΩ
- added U10: XL4015E1, EasyEDA:TO-263-5_L10.2-W8.9-P1.70-TL, symbol EasyEDA:XL4015E1
Connections:
- net ADXL_INT1: now also U1.86 (PD5); no longer U1.42 (PE11)
- net ADXL_INT2: now also U1.85 (PD4); no longer U1.41 (PE10)
- net BAT_LEVEL: now also U1.15 (PC0); no longer U1.97 (PE0)
- net BMI_GYRO_CS: now also U1.83 (PD2); no longer U1.81 (PD0)
- net BMI_GYRO_INT1: now also U1.66 (PC9); no longer U1.83 (PD2)
- net BMI_GYRO_INT2: now also U1.65 (PC8); no longer U1.84 (PD3)
- net BMI_accel_CS: now also U1.87 (PD6); no longer U1.85 (PD4)
- net BMI_accel_INT1: now also U1.81 (PD0); no longer U1.86 (PD5)
- net BMI_accel_INT2: now also U1.82 (PD1); no longer U1.87 (PD6)
- net GND: now also J1.1 (Pin_1), C2.2, C29.1, C3.2, C31.1, D7.1, J4.1 (Pin_1), J6.1 (Pin_1), R24.2, U10.1 (GND); no longer J1.2 (Pin_2)
- net LoRa_RST: now also U1.36 (PB1); no longer U1.43 (PE12)
- net MS5607_NSS: no longer U1.77 (PA15)
- net VBAT+: now also Pyro_CH1.1 (Pin_1), Pyro_CH2.2 (Pin_2), C19.2, C2.1, C29.2, J6.2 (Pin_2), U10.5 (VIN)
- net at D3.2: now also J1.2 (Pin_2); no longer J1.1 (Pin_1)
- net at Pyro_CH1.2 (Pin_2): now also Q1.7 (D1), Q1.8 (D1)
- net +5Vservo: now reaches SERVO1.2 (Pin_2), SERVO2.2 (Pin_2)
- net +5Vservo: now also C3.1, C31.2, J4.2 (Pin_2), L2.2, R8.2
- net MS5607_CS: now reaches U1.67 (PA8)
- net MS5607_SCLK: now reaches U1.68 (PA9)
- net ADXL_MISO: no longer names the net of U1.17 (PC2)
- net ADXL_MOSI renamed MS5607_MOSI
- net ADXL_NSS: no longer names the net of U1.51 (PB12)
- net ADXL_SCLK: no longer names the net of U1.47 (PB10)
- net DAT0: no longer names the net of U1.53 (PB14)
- net DAT1: no longer names the net of U1.54 (PB15)
- net DAT2: no longer names the net of U1.89 (PB3)
- net DAT3: no longer names the net of U1.90 (PB4)
- net DAT4: no longer names the net of U1.95 (PB8)
- net DAT5: no longer names the net of U1.96 (PB9)
- net DAT6: no longer names the net of U1.63 (PC6)
- net DAT7: no longer names the net of U1.64 (PC7)
- net RST_n: no longer names the net of U1.58 (PD11)
- net eMMC_CLK: no longer names the net of U1.16 (PC1)
- net eMMC_CMD: no longer names the net of U1.88 (PD7)
- new net: R24.1, R8.1, U10.2 (FB)
- new net: C19.1, U10.4 (VC)
- new net: D7.2, L2.1, U10.3 (SW), U10.6 (SW)
- new net ADXL_CS: U1.97 (PE0)
- new net MS5607_MISO: U1.84 (PD3)
- no-connect marks 25 -> 17
Other:
- note added: "5V Converter (Max 1A)"
- note removed: "Converter (Max 1A)"
- moved on the sheet: C17, LED3, R39

Commit message: 1
Connections:
- net eMMC_CLK: now reaches U1.16 (PC1)
- net DAT0: now reaches U1.53 (PB14)
- net DAT1: now reaches U1.54 (PB15)
- net eMMC_CMD: now reaches U1.88 (PD7)
- net DAT2: now reaches U1.89 (PB3)
- net DAT3: now reaches U1.90 (PB4)
Changed lines of the file:
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@@
 		)
 	)
+	(global_label "DAT0"
+		(shape bidirectional)
+		(at 104.14 116.84 0)
+		(fields_autoplaced yes)
+		(effects
+			(font
+				(size 1.27 1.27)
+			)
+			(justify left)
+		)
+		(property "Intersheetrefs" "${INTERSHEET_REFS}"
+			(at 112.7722 116.84 0)
+			(effects
+				(font
+					(size 1.27 1.27)
+				)
+				(justify left)
+				(hide yes)
+			)
+		)
+	)
 	(global_label "VBAT+"
 		(shape input)
@@
 		)
 	)
+	(global_label "DAT2"
+		(shape bidirectional)
+		(at 102.87 91.44 0)
+		(fields_autoplaced yes)
+		(effects
+			(font
+				(size 1.27 1.27)
+			)
+			(justify left)
+		)
+		(property "Intersheetrefs" "${INTERSHEET_REFS}"
+			(at 111.5022 91.44 0)
+			(effects
+				(font
+					(size 1.27 1.27)
+				)
+				(justify left)
+				(hide yes)
+			)
+		)
+	)
 	(global_label "PYRO_A"
 		(shape input)
@@
 		)
 	)
+	(global_label "DAT3"
+		(shape bidirectional)
+		(at 102.87 93.98 0)
+		(fields_autoplaced yes)
+		(effects
+			(font
+				(size 1.27 1.27)
+			)
+			(justify left)
+		)
+		(property "Intersheetrefs" "${INTERSHEET_REFS}"
+			(at 111.5022 93.98 0)
+			(effects
+				(font
+					(size 1.27 1.27)
+				)
+				(justify left)
+				(hide yes)
+			)
+		)
+	)
 	(global_label "PYRO_A"
 		(shape output)
@@
 		)
 	)
+	(global_label "DAT1"
+		(shape bidirectional)
+		(at 104.14 119.38 0)
+		(fields_autoplaced yes)
+		(effects
+			(font
+				(size 1.27 1.27)
+			)
+			(justify left)
+		)
+		(property "Intersheetrefs" "${INTERSHEET_REFS}"
+			(at 112.7722 119.38 0)
+			(effects
+				(font
+					(size 1.27 1.27)
+				)
+				(justify left)
+				(hide yes)
+			)
+		)
+	)
 	(global_label "SWDIO"
 		(shape bidirectional)
@@
 		)
 	)
+	(global_label "eMMC_CLK"
+		(shape output)
+		(at 102.87 127 0)
+		(fields_autoplaced yes)
+		(effects
+			(font
+				(size 1.27 1.27)
+			)
+			(justify left)
+		)
+		(property "Intersheetrefs" "${INTERSHEET_REFS}"
+			(at 115.6523 127 0)
+			(effects
+				(font
+					(size 1.27 1.27)
+				)
+				(justify left)
+				(hide yes)
+			)
+		)
+	)
 	(global_label "PWM_A"
 		(shape input)
@@
 		)
 	)
+	(global_label "eMMC_CMD"
+		(shape bidirectional)
+		(at 57.15 124.46 180)
+		(fields_autoplaced yes)
+		(effects
+			(font
+				(size 1.27 1.27)
+			)
+			(justify right)
+		)
+		(property "Intersheetrefs" "${INTERSHEET_REFS}"
+			(at 42.8331 124.46 0)
+			(effects
+				(font
+					(size 1.27 1.27)
+				)
+				(justify right)
+				(hide yes)
+			)
+		)
+	)
 	(global_label "nRST"
 		(shape input)
@@
 		(on_board yes)
 		(dnp no)
-		(fields_autoplaced yes)
 		(property "Reference" "LED3"
 			(at 172.72 253.9046 0)
@@
 		)
 		(property "Digikey Parts" "B1911USD-20D000114U1930"
-			(at 170.18 255.27 0)
+			(at 148.336 255.016 0)
 			(effects
 				(font
@@
 		)
 		(property "Digikey Parts" "RC0603JR-071KL"
-			(at 170.18 270.51 0)
+			(at 154.686 270.51 0)
 			(effects
 				(font

Commit message: .
Parts:
- added C35: 180uF, 180uF:CAP_FKS_F_PAN, symbol Device:C_Small
- added C37: 1uF, PCM_JLCPCB:C_0603, symbol PCM_JLCPCB-Capacitors:0402,1uF
- added C38: 470uF, Capacitor_SMD:CP_Elec_8x10, symbol PCM_JLCPCB-Capacitors:Plugin,D10xL16mm,470uF
- added D8: SS34_C466502, GNSS:DIOM7959X262N, symbol EasyEDA:SS34_C466502
- added L3: 68uH, EasyEDA:IND-SMD_L22.5-W22.0, symbol Device:L
- added U7: XL1509-5.0, Package_SO:SOIC-8_3.9x4.9mm_P1.27mm, symbol Regulator_Switching:XL1509-5.0
Connections:
- net +5V: now also C35.1, D8.1, L3.2, U7.3 (FB)
- net GND: now also C35.2, C37.2, C38.2, D8.2, U7.5 (GND), U7.6 (GND), U7.7 (GND), U7.8 (GND)
- net VBAT+: now also C37.1, C38.1, U7.1 (VIN)
- new net: L3.1, U7.2 (OUT)
Other:
- moved on the sheet: C20, C23, C25, L1, R10, U8

Commit message: ..
Connections:
- net GNSS_SAFEBOOT: now also U1.13 (PH1); no longer U1.44 (PE13)
- no-connect marks 17 -> 16
Other:
- moved on the sheet: J2
Changed lines of the file:
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@@
 	(text "place jumper cap"
 		(exclude_from_sim no)
-		(at 29.21 58.42 90)
+		(at 30.734 62.738 0)
 		(effects
 			(font
@@
 	)
 	(junction
+		(at 39.37 58.42)
+		(diameter 0)
+		(color 0 0 0 0)
+	)
+	(junction
 		(at 203.2 31.75)
 		(diameter 0)
@@
 	)
 	(junction
-		(at 44.45 58.42)
-		(diameter 0)
-		(color 0 0 0 0)
-	)
-	(junction
 		(at 303.53 100.33)
 		(diameter 0)
@@
 	)
 	(no_connect
-		(at 57.15 55.88)
-	)
-	(no_connect
 		(at 205.74 140.97)
 	)
@@
 	(wire
 		(pts
-			(xy 38.1 58.42) (xy 44.45 58.42)
+			(xy 33.02 58.42) (xy 39.37 58.42)
 		)
 		(stroke
@@
 	(wire
 		(pts
-			(xy 44.45 58.42) (xy 44.45 71.12)
+			(xy 39.37 58.42) (xy 39.37 71.12)
 		)
 		(stroke
@@
 	(wire
 		(pts
+			(xy 39.37 58.42) (xy 44.45 58.42)
+		)
+		(stroke
+			(width 0)
+			(type default)
+		)
+	)
+	(wire
+		(pts
 			(xy 271.78 193.04) (xy 271.78 201.93)
 		)
@@
 	(wire
 		(pts
-			(xy 40.64 52.07) (xy 40.64 55.88)
+			(xy 35.56 52.07) (xy 35.56 55.88)
 		)
 		(stroke
@@
 	(wire
 		(pts
-			(xy 40.64 55.88) (xy 38.1 55.88)
+			(xy 35.56 55.88) (xy 33.02 55.88)
 		)
 		(stroke
@@
 	(wire
 		(pts
+			(xy 55.88 55.88) (xy 57.15 55.88)
+		)
+		(stroke
+			(width 0)
+			(type default)
+		)
+	)
+	(wire
+		(pts
 			(xy 368.3 194.31) (xy 368.3 199.39)
 		)
@@
 	(wire
 		(pts
-			(xy 38.1 60.96) (xy 40.64 60.96)
+			(xy 33.02 60.96) (xy 35.56 60.96)
 		)
 		(stroke
@@
 	(wire
 		(pts
-			(xy 40.64 60.96) (xy 40.64 62.23)
+			(xy 35.56 60.96) (xy 35.56 62.23)
 		)
 		(stroke
@@
 	(wire
 		(pts
-			(xy 52.07 96.52) (xy 57.15 96.52)
-		)
-		(stroke
-			(width 0)
-			(type default)
-		)
-	)
-	(wire
-		(pts
 			(xy 121.92 205.74) (xy 121.92 203.2)
 		)
@@
 	(global_label "BOOT0"
 		(shape input)
-		(at 44.45 71.12 270)
+		(at 39.37 71.12 270)
 		(fields_autoplaced yes)
 		(effects
@@
 		)
 		(property "Intersheetrefs" "${INTERSHEET_REFS}"
-			(at 44.45 80.2133 90)
+			(at 39.37 80.2133 90)
 			(effects
 				(font
@@
 	(global_label "GNSS_SAFEBOOT"
 		(shape output)
-		(at 52.07 96.52 180)
+		(at 55.88 55.88 180)
 		(fields_autoplaced yes)
 		(effects
@@
 		)
 		(property "Intersheetrefs" "${INTERSHEET_REFS}"
-			(at 33.6634 96.52 0)
+			(at 37.4734 55.88 0)
 			(effects
 				(font
@@
 	(symbol
 		(lib_id "power:GND")
-		(at 40.64 62.23 0)
+		(at 35.56 62.23 0)
 		(unit 1)
 		(exclude_from_sim no)
@@
 		(fields_autoplaced yes)
 		(property "Reference" "#PWR0107"
-			(at 40.64 68.58 0)
+			(at 35.56 68.58 0)
 			(effects
 				(font
@@
 		)
 		(property "Value" "GND"
-			(at 40.64 67.31 0)
+			(at 35.56 67.31 0)
 			(effects
 				(font
@@
 		)
 		(property "Footprint" ""
-			(at 40.64 62.23 0)
+			(at 35.56 62.23 0)
 			(effects
 				(font
@@
 		)
 		(property "Datasheet" ""
-			(at 40.64 62.23 0)
+			(at 35.56 62.23 0)
 			(effects
 				(font
@@
 		)
 		(property "Description" "Power symbol creates a global label with name \"GND\" , ground"
-			(at 40.64 62.23 0)
+			(at 35.56 62.23 0)
 			(effects
 				(font
@@
 	(symbol
 		(lib_id "power:+3.3V")
-		(at 40.64 52.07 0)
+		(at 35.56 52.07 0)
 		(unit 1)
 		(exclude_from_sim no)
@@
 		(fields_autoplaced yes)
 		(property "Reference" "#PWR029"
-			(at 40.64 55.88 0)
+			(at 35.56 55.88 0)
 			(effects
 				(font
@@
 		)
 		(property "Value" "+3.3V"
-			(at 40.64 46.99 0)
+			(at 35.56 46.99 0)
 			(effects
 				(font
@@
 		)
 		(property "Footprint" ""
-			(at 40.64 52.07 0)
+			(at 35.56 52.07 0)
 			(effects
 				(font
@@
 		)
 		(property "Datasheet" ""
-			(at 40.64 52.07 0)
+			(at 35.56 52.07 0)
 			(effects
 				(font
@@
 		)
 		(property "Description" "Power symbol creates a global label with name \"+3.3V\""
-			(at 40.64 52.07 0)
+			(at 35.56 52.07 0)
 			(effects
 				(font
@@
 		(dnp no)
 		(property "Reference" "R9"
-			(at 48.26 56.388 90)
+			(at 43.942 60.452 90)
 			(effects
 				(font
@@
 	(symbol
 		(lib_id "Connector:Conn_01x03_Pin")
-		(at 33.02 58.42 0)
+		(at 27.94 58.42 0)
 		(unit 1)
 		(exclude_from_sim no)
@@
 		(dnp no)
 		(property "Reference" "J2"
-			(at 30.734 58.42 90)
+			(at 25.654 58.42 90)
 			(effects
 				(font
@@
 		)
 		(property "Value" "BOOT0"
-			(at 31.75 58.42 90)
+			(at 26.67 58.42 90)
 			(effects
 				(font
@@
 		)
 		(property "Footprint" "Connector_PinHeader_2.54mm:PinHeader_1x03_P2.54mm_Vertical"
-			(at 33.02 58.42 0)
+			(at 27.94 58.42 0)
 			(effects
 				(font
@@
 		)
 		(property "Datasheet" "~"
-			(at 33.02 58.42 0)
+			(at 27.94 58.42 0)
 			(effects
 				(font
@@
 		)
 		(property "Description" "Generic connector, single row, 01x03, script generated"
-			(at 33.02 58.42 0)
+			(at 27.94 58.42 0)
 			(effects
 				(font
@@
 		)
 		(property "DC Resistance (DCR)" ""
-			(at 33.02 58.42 0)
+			(at 27.94 58.42 0)
 			(effects
 				(font
@@
 		)
 		(property "Equivalent Series Resistance(ESR)" ""
-			(at 33.02 58.42 0)
+			(at 27.94 58.42 0)
 			(effects
 				(font
@@
 		)
 		(property "Frequency - Self Resonant" ""
-			(at 33.02 58.42 0)
+			(at 27.94 58.42 0)
 			(effects
 				(font
@@
 		)
 		(property "Inductance" ""
-			(at 33.02 58.42 0)
+			(at 27.94 58.42 0)
 			(effects
 				(font
@@
 		)
 		(property "Operating Temperature" ""
-			(at 33.02 58.42 0)
+			(at 27.94 58.42 0)
 			(effects
 				(font
@@
 		)
 		(property "Q @ Freq" ""
-			(at 33.02 58.42 0)
+			(at 27.94 58.42 0)
 			(effects
 				(font
@@
 		)
 		(property "Rated Current" ""
-			(at 33.02 58.42 0)
+			(at 27.94 58.42 0)
 			(effects
 				(font
@@
 		)
 		(property "Rated Voltage" ""
-			(at 33.02 58.42 0)
+			(at 27.94 58.42 0)
 			(effects
 				(font
@@
 		)
 		(property "Sim.Pins" ""
-			(at 33.02 58.42 0)
+			(at 27.94 58.42 0)
 			(effects
 				(font
@@
 		)
 		(property "Digikey Parts" ""
-			(at 33.02 58.42 0)
+			(at 27.94 58.42 0)
 			(effects
 				(font

Commit message: ......
Parts:
- C35: footprint 180uF:CAP_FKS_F_PAN -> Capacitor_SMD:CP_Elec_5x5.3
- C38: value 470uF -> 100uF; footprint Capacitor_SMD:CP_Elec_8x10 -> Capacitor_SMD:CP_Elec_5x5.3; Digikey UUD1C471MNL1GS -> EEE-1AA101WR
- L3: value 68uH -> 33uH; footprint EasyEDA:IND-SMD_L22.5-W22.0 -> Inductor_SMD:L_Bourns_SRP1038C_10.0x10.0mm; Digikey Parts CSBX2212-680M -> 1274AS-H-330M=P3
Connections:
- net +5V: no longer D8.1
- net at L3.1, U7.2 (OUT): now also D8.1
Other:
- moved on the sheet: C37, D8

Commit message: fkdjgfg
Parts:
- L1: footprint EasyEDA:IND-SMD_L4.0-W4.0_XFL4020-102MEB -> newinductor:IND_EPCOS_B82432T_EPC; Digikey Parts CS160808-2R2K -> B82432T1222K000
Changed lines of the file:
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@@
 			)
 		)
-		(property "Footprint" "EasyEDA:IND-SMD_L4.0-W4.0_XFL4020-102MEB"
+		(property "Footprint" "newinductor:IND_EPCOS_B82432T_EPC"
 			(at 505.46 111.76 0)
 			(effects
@@
 			)
 		)
-		(property "Digikey Parts" "CS160808-2R2K"
+		(property "Digikey Parts" "B82432T1222K000"
 			(at 505.206 105.918 0)
 			(effects

Commit message: Feat: Minor improvement
Parts:
- removed R22, R39: 1kΩ, PCM_JLCPCB:R_0603, symbol PCM_JLCPCB-Resistors:0402,1kΩ
- added R22, R36: 470Ω, PCM_JLCPCB:R_0603, symbol PCM_JLCPCB-Resistors:0402,470Ω
Connections:
- net GND: now also R22.2, R36.2
- net at LED3.1: now also R36.1
- net at PB0.1: now also R22.1
Other:
- moved on the sheet: C20, C23, C25, L1, PB0, R10, U8
