File: untitled.kicad_sch (KiCad schematic)
At the start: 4 parts

Commit message: Chore: push new design
Parts:
- C27, C34: footprint PCM_JLCPCB:C_0402 -> PCM_JLCPCB:C_0603
Connections:
- net DIO1 renamed LORA_DIO1
- net LORA_DIO3: no longer names the net of U15.11 (DIO3)
- no-connect marks 0 -> 1

Commit message: Special version
Parts:
- C27: Digikey Parts (none) -> CL10B104KA8NNNC
- C34: Digikey Parts (none) -> CL10A106KP8NNNC
Changed lines of the file:
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@@
+			)
+		)
+		(property "Digikey Parts" "CL10B104KA8NNNC"
+			(at 81.28 100.33 0)
+			(effects
+				(font
+					(size 1.27 1.27)
+				)
 			)
 		)
@@
 		)
 		(property "Sim.Pins" ""
+			(at 63.5 100.33 0)
+			(effects
+				(font
+					(size 1.27 1.27)
+				)
+			)
+		)
+		(property "Digikey Parts" "CL10A106KP8NNNC"
 			(at 63.5 100.33 0)
 			(effects
@@
 			)
 		)
+		(property "Digikey Parts" ""
+			(at 77.47 73.66 0)
+			(effects
+				(font
+					(size 1.27 1.27)
+				)
+			)
+		)
 		(pin "5"
 		)
@@
 			(at 120.65 69.85 0)
 			(effects
+				(font
+					(size 1.27 1.27)
+				)
+			)
+		)
+		(property "Digikey Parts" ""
+			(at 120.65 69.85 0)
+			(effects

Commit message: Complete Redesign
Parts:
- added J7: U.FL, PCM_JLCPCB:IPEX-SMD_BWIPX-1-001E, symbol PCM_JLCPCB-Extended:RF, Connector, U.FL
Connections:
- net GND: now also J7.2 (Ext), J7.3; no longer RF1.2, RF1.3, RF1.4, RF1.5
- net at U15.9 (ANT): now also J7.1 (In); no longer RF1.1
Other:
- moved on the sheet: RF1

Commit message: 1
Parts:
- removed J7: U.FL, PCM_JLCPCB:IPEX-SMD_BWIPX-1-001E, symbol PCM_JLCPCB-Extended:RF, Connector, U.FL
Connections:
- net GND: now also RF1.2, RF1.3, RF1.4, RF1.5
- net at U15.9 (ANT): now also RF1.1
Other:
- moved on the sheet: RF1
